File: Auralab_Workstation/pcbwaycontest.kicad_sch (KiCad schematic)
At the start: 12 parts, among them J1 Conn_Coaxial, Q1 BS170, SW1 SW_SPDT, U1 TL072, U2 MCP3201, U3 REF3033, U4 INA226

Commit message: Add files via upload
Connections:
- net at U3.2 (OUT): now also U2.1 (Vref)
- net at U1.1: now also D1.1 (K)
- net at SW1.3 (C): now also C1.2, R1.1
- net at R2.1: now also Q1.3 (S), U4.9 (Vin-)
- net at R2.2: now also Q1.2 (G)
- net at R3.1: now also R1.2
- net at U4.10 (Vin+): now also U4.8 (Vbus)
- net I2C_SDA: now reaches U4.4 (SDA)
- net I2C_SCL: now reaches U4.5 (SCL)
Other:
- moved on the sheet: Q1, R2

Commit message: Add files via upload
Connections:
- net +3V3_DIGITAL: now reaches U3.1 (IN)
- net +3V3_DIGITAL: now also U2.8 (Vdd)
- net GNDA: now reaches U3.3 (GND)
- net GNDA: now also D1.2 (A), J1.2 (Ext), R3.2, U2.3 (IN-), U2.4 (Vss)
- net at D1.1 (K), U1.1: now also U1.2 (-), U2.2 (IN+)
- net at U1.3 (+): now also R1.2, R3.1
- net ADC_CS: now reaches U2.5 (~{CS}/SHDN)
- net ADC_MISO: now reaches U2.6 (Dout)
- net ADC_SCLK: now reaches U2.7 (CLK)
- net GND: now reaches U4.6 (VS)
- net GND: now also U4.7 (GND)
- net RANGE_SELECT: now reaches Q1.1 (D)

Commit message: just rotated one net label in ur sch
Changed lines of the file:
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@@
 	(global_label "+3V3_DIGITAL"
 		(shape bidirectional)
-		(at 147.32 66.04 90)
+		(at 147.32 66.04 0)
 		(fields_autoplaced yes)
 		(effects
@@
 		)
 		(property "Intersheetrefs" "${INTERSHEET_REFS}"
-			(at 147.32 49.062 90)
+			(at 164.298 66.04 0)
 			(effects
 				(font
@@
 		(dnp no)
 		(fields_autoplaced yes)
-		(property "Reference" "U3"
+		(property "Reference" "U?"
 			(at 143.51 72.3899 0)
 			(effects
@@
 				)
 			)
+			(project "Auralab_Workstation"
+				(path "/db223ba7-bea5-428e-a07f-3236299d6518/15949506-3bc7-4c2f-a211-94c4f1c42d64"
+					(reference "U?")
+					(unit 1)
+				)
+			)
 		)
 	)
@@
 		(dnp no)
 		(fields_autoplaced yes)
-		(property "Reference" "U1"
+		(property "Reference" "U?"
 			(at 119.38 88.9 0)
 			(effects
@@
 				)
 			)
+			(project "Auralab_Workstation"
+				(path "/db223ba7-bea5-428e-a07f-3236299d6518/15949506-3bc7-4c2f-a211-94c4f1c42d64"
+					(reference "U?")
+					(unit 1)
+				)
+			)
 		)
 	)
@@
 		(dnp no)
 		(fields_autoplaced yes)
-		(property "Reference" "SW1"
+		(property "Reference" "SW?"
 			(at 68.58 104.14 0)
 			(effects
@@
 				)
 			)
+			(project "Auralab_Workstation"
+				(path "/db223ba7-bea5-428e-a07f-3236299d6518/15949506-3bc7-4c2f-a211-94c4f1c42d64"
+					(reference "SW?")
+					(unit 1)
+				)
+			)
 		)
 	)
@@
 		(dnp no)
 		(fields_autoplaced yes)
-		(property "Reference" "R2"
+		(property "Reference" "R?"
 			(at 59.69 163.8299 0)
 			(effects
@@
 				)
 			)
+			(project "Auralab_Workstation"
+				(path "/db223ba7-bea5-428e-a07f-3236299d6518/15949506-3bc7-4c2f-a211-94c4f1c42d64"
+					(reference "R?")
+					(unit 1)
+				)
+			)
 		)
 	)
@@
 		(dnp no)
 		(fields_autoplaced yes)
-		(property "Reference" "J1"
+		(property "Reference" "J?"
 			(at 46.99 82.8431 0)
 			(effects
@@
 				)
 			)
+			(project "Auralab_Workstation"
+				(path "/db223ba7-bea5-428e-a07f-3236299d6518/15949506-3bc7-4c2f-a211-94c4f1c42d64"
+					(reference "J?")
+					(unit 1)
+				)
+			)
 		)
 	)
@@
 		(dnp no)
 		(fields_autoplaced yes)
-		(property "Reference" "R3"
+		(property "Reference" "R?"
 			(at 127 116.8399 0)
 			(effects
@@
 				)
 			)
+			(project "Auralab_Workstation"
+				(path "/db223ba7-bea5-428e-a07f-3236299d6518/15949506-3bc7-4c2f-a211-94c4f1c42d64"
+					(reference "R?")
+					(unit 1)
+				)
+			)
 		)
 	)
@@
 		(dnp no)
 		(fields_autoplaced yes)
-		(property "Reference" "U2"
+		(property "Reference" "U?"
 			(at 124.0633 59.69 0)
 			(effects
@@
 				)
 			)
+			(project "Auralab_Workstation"
+				(path "/db223ba7-bea5-428e-a07f-3236299d6518/15949506-3bc7-4c2f-a211-94c4f1c42d64"
+					(reference "U?")
+					(unit 1)
+				)
+			)
 		)
 	)
@@
 		(dnp no)
 		(fields_autoplaced yes)
-		(property "Reference" "R1"
+		(property "Reference" "R?"
 			(at 95.25 110.4899 0)
 			(effects
@@
 				)
 			)
+			(project "Auralab_Workstation"
+				(path "/db223ba7-bea5-428e-a07f-3236299d6518/15949506-3bc7-4c2f-a211-94c4f1c42d64"
+					(reference "R?")
+					(unit 1)
+				)
+			)
 		)
 	)
@@
 		(dnp no)
 		(fields_autoplaced yes)
-		(property "Reference" "U4"
+		(property "Reference" "U?"
 			(at 82.1533 133.35 0)
 			(effects
@@
 				)
 			)
+			(project "Auralab_Workstation"
+				(path "/db223ba7-bea5-428e-a07f-3236299d6518/15949506-3bc7-4c2f-a211-94c4f1c42d64"
+					(reference "U?")
+					(unit 1)
+				)
+			)
 		)
 	)
@@
 		(dnp no)
 		(fields_autoplaced yes)
-		(property "Reference" "Q1"
+		(property "Reference" "Q?"
 			(at 120.65 157.4799 0)
 			(effects
@@
 				)
 			)
+			(project "Auralab_Workstation"
+				(path "/db223ba7-bea5-428e-a07f-3236299d6518/15949506-3bc7-4c2f-a211-94c4f1c42d64"
+					(reference "Q?")
+					(unit 1)
+				)
+			)
 		)
 	)
@@
 		(dnp no)
 		(fields_autoplaced yes)
-		(property "Reference" "C1"
+		(property "Reference" "C?"
 			(at 96.52 78.7399 0)
 			(effects
@@
 				)
 			)
+			(project "Auralab_Workstation"
+				(path "/db223ba7-bea5-428e-a07f-3236299d6518/15949506-3bc7-4c2f-a211-94c4f1c42d64"
+					(reference "C?")
+					(unit 1)
+				)
+			)
 		)
 	)
@@
 		(dnp no)
 		(fields_autoplaced yes)
-		(property "Reference" "D1"
+		(property "Reference" "D?"
 			(at 73.66 55.88 0)
 			(effects
@@
 					(unit 1)
 				)
+			)
+			(project "Auralab_Workstation"
+				(path "/db223ba7-bea5-428e-a07f-3236299d6518/15949506-3bc7-4c2f-a211-94c4f1c42d64"
+					(reference "D?")
+					(unit 1)
+				)

Commit message: Add files via upload
Connections:
- net GND: now also U4.1 (A1), U4.2 (A0)
- net CURRENT_IN: now reaches U4.10 (Vin+), U4.8 (Vbus)
- net CURRENT_ALERT: now reaches U4.3 (~{Alert})
Changed lines of the file:
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@@
+	)
+	(junction
+		(at 62.23 146.05)
+		(diameter 0)
+		(color 0 0 0 0)
 	)
 	(junction
@@
 	(wire
 		(pts
+			(xy 58.42 146.05) (xy 62.23 146.05)
+		)
+		(stroke
+			(width 0)
+			(type default)
+		)
+	)
+	(wire
+		(pts
 			(xy 92.71 115.57) (xy 92.71 121.92)
 		)
@@
 	(wire
 		(pts
+			(xy 90.17 156.21) (xy 92.71 156.21)
+		)
+		(stroke
+			(width 0)
+			(type default)
+		)
+	)
+	(wire
+		(pts
 			(xy 127 72.39) (xy 102.87 72.39)
 		)
@@
 	(wire
 		(pts
-			(xy 62.23 140.97) (xy 62.23 151.13)
+			(xy 62.23 140.97) (xy 62.23 146.05)
+		)
+		(stroke
+			(width 0)
+			(type default)
+		)
+	)
+	(wire
+		(pts
+			(xy 62.23 146.05) (xy 62.23 151.13)
 		)
 		(stroke
@@
 			(width 0)
 			(type default)
+		)
+	)
+	(label "CURRENT_ALERT"
+		(at 92.71 156.21 0)
+		(effects
+			(font
+				(size 1.27 1.27)
+			)
+			(justify left bottom)
 		)
 	)
@@
 		)
 	)
+	(global_label "CURRENT_IN"
+		(shape bidirectional)
+		(at 58.42 146.05 180)
+		(fields_autoplaced yes)
+		(effects
+			(font
+				(size 1.27 1.27)
+			)
+			(justify right)
+		)
+		(property "Intersheetrefs" "${INTERSHEET_REFS}"
+			(at 42.833 146.05 0)
+			(effects
+				(font
+					(size 1.27 1.27)
+				)
+				(justify right)
+				(hide yes)
+			)
+		)
+	)
 	(global_label "GND"
 		(shape bidirectional)
@@
 		)
 	)
+	(global_label "GND"
+		(shape bidirectional)
+		(at 90.17 143.51 0)
+		(fields_autoplaced yes)
+		(effects
+			(font
+				(size 1.27 1.27)
+			)
+			(justify left)
+		)
+		(property "Intersheetrefs" "${INTERSHEET_REFS}"
+			(at 98.137 143.51 0)
+			(effects
+				(font
+					(size 1.27 1.27)
+				)
+				(justify left)
+				(hide yes)
+			)
+		)
+	)
 	(global_label "I2C_SDA"
 		(shape bidirectional)
@@
 		)
 	)
+	(global_label "GND"
+		(shape bidirectional)
+		(at 90.17 140.97 0)
+		(fields_autoplaced yes)
+		(effects
+			(font
+				(size 1.27 1.27)
+			)
+			(justify left)
+		)
+		(property "Intersheetrefs" "${INTERSHEET_REFS}"
+			(at 98.137 140.97 0)
+			(effects
+				(font
+					(size 1.27 1.27)
+				)
+				(justify left)
+				(hide yes)
+			)
+		)
+	)
 	(global_label "ADC_MISO"
 		(shape bidirectional)
@@
 	(global_label "+3V3_DIGITAL"
 		(shape bidirectional)
-		(at 147.32 66.04 0)
+		(at 147.32 66.04 90)
 		(fields_autoplaced yes)
 		(effects
@@
 		)
 		(property "Intersheetrefs" "${INTERSHEET_REFS}"
-			(at 164.298 66.04 0)
+			(at 147.32 49.062 90)
 			(effects
 				(font
@@
 		(dnp no)
 		(fields_autoplaced yes)
-		(property "Reference" "U?"
+		(property "Reference" "U3"
 			(at 143.51 72.3899 0)
 			(effects
@@
 				(path "/0cb921c9-5493-42a4-9366-73ecb4110608"
 					(reference "U3")
-					(unit 1)
-				)
-			)
-			(project "Auralab_Workstation"
-				(path "/db223ba7-bea5-428e-a07f-3236299d6518/15949506-3bc7-4c2f-a211-94c4f1c42d64"
-					(reference "U?")
 					(unit 1)
 				)
@@
 		(dnp no)
 		(fields_autoplaced yes)
-		(property "Reference" "U?"
+		(property "Reference" "U1"
 			(at 119.38 88.9 0)
 			(effects
@@
 				(path "/0cb921c9-5493-42a4-9366-73ecb4110608"
 					(reference "U1")
-					(unit 1)
-				)
-			)
-			(project "Auralab_Workstation"
-				(path "/db223ba7-bea5-428e-a07f-3236299d6518/15949506-3bc7-4c2f-a211-94c4f1c42d64"
-					(reference "U?")
 					(unit 1)
 				)
@@
 		(dnp no)
 		(fields_autoplaced yes)
-		(property "Reference" "SW?"
+		(property "Reference" "SW1"
 			(at 68.58 104.14 0)
 			(effects
@@
 				(path "/0cb921c9-5493-42a4-9366-73ecb4110608"
 					(reference "SW1")
-					(unit 1)
-				)
-			)
-			(project "Auralab_Workstation"
-				(path "/db223ba7-bea5-428e-a07f-3236299d6518/15949506-3bc7-4c2f-a211-94c4f1c42d64"
-					(reference "SW?")
 					(unit 1)
 				)
@@
 		(dnp no)
 		(fields_autoplaced yes)
-		(property "Reference" "R?"
+		(property "Reference" "R2"
 			(at 59.69 163.8299 0)
 			(effects
@@
 				(path "/0cb921c9-5493-42a4-9366-73ecb4110608"
 					(reference "R2")
-					(unit 1)
-				)
-			)
-			(project "Auralab_Workstation"
-				(path "/db223ba7-bea5-428e-a07f-3236299d6518/15949506-3bc7-4c2f-a211-94c4f1c42d64"
-					(reference "R?")
 					(unit 1)
 				)
@@
 		(dnp no)
 		(fields_autoplaced yes)
-		(property "Reference" "J?"
+		(property "Reference" "J1"
 			(at 46.99 82.8431 0)
 			(effects
@@
 				(path "/0cb921c9-5493-42a4-9366-73ecb4110608"
 					(reference "J1")
-					(unit 1)
-				)
-			)
-			(project "Auralab_Workstation"
-				(path "/db223ba7-bea5-428e-a07f-3236299d6518/15949506-3bc7-4c2f-a211-94c4f1c42d64"
-					(reference "J?")
 					(unit 1)
 				)
@@
 		(dnp no)
 		(fields_autoplaced yes)
-		(property "Reference" "R?"
+		(property "Reference" "R3"
 			(at 127 116.8399 0)
 			(effects
@@
 				(path "/0cb921c9-5493-42a4-9366-73ecb4110608"
 					(reference "R3")
-					(unit 1)
-				)
-			)
-			(project "Auralab_Workstation"
-				(path "/db223ba7-bea5-428e-a07f-3236299d6518/15949506-3bc7-4c2f-a211-94c4f1c42d64"
-					(reference "R?")
 					(unit 1)
 				)
@@
 		(dnp no)
 		(fields_autoplaced yes)
-		(property "Reference" "U?"
+		(property "Reference" "U2"
 			(at 124.0633 59.69 0)
 			(effects
@@
 				(path "/0cb921c9-5493-42a4-9366-73ecb4110608"
 					(reference "U2")
-					(unit 1)
-				)
-			)
-			(project "Auralab_Workstation"
-				(path "/db223ba7-bea5-428e-a07f-3236299d6518/15949506-3bc7-4c2f-a211-94c4f1c42d64"
-					(reference "U?")
 					(unit 1)
 				)
@@
 		(dnp no)
 		(fields_autoplaced yes)
-		(property "Reference" "R?"
+		(property "Reference" "R1"
 			(at 95.25 110.4899 0)
 			(effects
@@
 				(path "/0cb921c9-5493-42a4-9366-73ecb4110608"
 					(reference "R1")
-					(unit 1)
-				)
-			)
-			(project "Auralab_Workstation"
-				(path "/db223ba7-bea5-428e-a07f-3236299d6518/15949506-3bc7-4c2f-a211-94c4f1c42d64"
-					(reference "R?")
 					(unit 1)
 				)
@@
 		(dnp no)
 		(fields_autoplaced yes)
-		(property "Reference" "U?"
+		(property "Reference" "U4"
 			(at 82.1533 133.35 0)
 			(effects
@@
 				(path "/0cb921c9-5493-42a4-9366-73ecb4110608"
 					(reference "U4")
-					(unit 1)
-				)
-			)
-			(project "Auralab_Workstation"
-				(path "/db223ba7-bea5-428e-a07f-3236299d6518/15949506-3bc7-4c2f-a211-94c4f1c42d64"
-					(reference "U?")
 					(unit 1)
 				)
@@
 		(dnp no)
 		(fields_autoplaced yes)
-		(property "Reference" "Q?"
+		(property "Reference" "Q1"
 			(at 120.65 157.4799 0)
 			(effects
@@
 				(path "/0cb921c9-5493-42a4-9366-73ecb4110608"
 					(reference "Q1")
-					(unit 1)
-				)
-			)
-			(project "Auralab_Workstation"
-				(path "/db223ba7-bea5-428e-a07f-3236299d6518/15949506-3bc7-4c2f-a211-94c4f1c42d64"
-					(reference "Q?")
 					(unit 1)
 				)
@@
 		(dnp no)
 		(fields_autoplaced yes)
-		(property "Reference" "C?"
+		(property "Reference" "C1"
 			(at 96.52 78.7399 0)
 			(effects
@@
 				(path "/0cb921c9-5493-42a4-9366-73ecb4110608"
 					(reference "C1")
-					(unit 1)
-				)
-			)
-			(project "Auralab_Workstation"
-				(path "/db223ba7-bea5-428e-a07f-3236299d6518/15949506-3bc7-4c2f-a211-94c4f1c42d64"
-					(reference "C?")
 					(unit 1)
 				)
@@
 		(dnp no)
 		(fields_autoplaced yes)
-		(property "Reference" "D?"
+		(property "Reference" "D1"
 			(at 73.66 55.88 0)
 			(effects
@@
 					(unit 1)
 				)
-			)
-			(project "Auralab_Workstation"
-				(path "/db223ba7-bea5-428e-a07f-3236299d6518/15949506-3bc7-4c2f-a211-94c4f1c42d64"
-					(reference "D?")
-					(unit 1)
-				)
