File: Auralab_Workstation/pcbwaycontest.kicad_sch (KiCad schematic)
At the start: 12 parts, among them J1 Conn_Coaxial, Q1 BS170, SW1 SW_SPDT, U1 TL072, U2 MCP3201, U3 REF3033, U4 INA226

Commit message: Made few changes in IN2A66 in urs
Parts:
- added R4: 0.1 Ohm, symbol Device:R
- R2: value R -> 10 Ohm
Connections:
- net CURRENT_IN: now also R2.1, R4.1
- net RANGE_SELECT: now also Q1.2 (G); no longer Q1.1 (D)
- net at Q1.3 (S), U4.9 (Vin-): now also R4.2; no longer R2.1
- net at R2.2: now also Q1.1 (D); no longer Q1.2 (G)
Other:
- moved on the sheet: Q1, R2
Changed lines of the file:
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@@
-	)
-	(junction
-		(at 67.31 153.67)
-		(diameter 0)
-		(color 0 0 0 0)
 	)
 	(junction
@@
 	)
 	(junction
+		(at 62.23 151.13)
+		(diameter 0)
+		(color 0 0 0 0)
+	)
+	(junction
 		(at 127 99.06)
 		(diameter 0)
@@
 		(color 0 0 0 0)
 	)
+	(junction
+		(at 52.07 151.13)
+		(diameter 0)
+		(color 0 0 0 0)
+	)
+	(junction
+		(at 52.07 170.18)
+		(diameter 0)
+		(color 0 0 0 0)
+	)
 	(wire
 		(pts
@@
 	(wire
 		(pts
+			(xy 52.07 170.18) (xy 52.07 168.91)
+		)
+		(stroke
+			(width 0)
+			(type default)
+		)
+	)
+	(wire
+		(pts
 			(xy 92.71 104.14) (xy 92.71 107.95)
 		)
@@
 	(wire
 		(pts
+			(xy 52.07 151.13) (xy 62.23 151.13)
+		)
+		(stroke
+			(width 0)
+			(type default)
+		)
+	)
+	(wire
+		(pts
 			(xy 124.46 111.76) (xy 124.46 114.3)
 		)
@@
 	(wire
 		(pts
+			(xy 25.4 152.4) (xy 25.4 151.13)
+		)
+		(stroke
+			(width 0)
+			(type default)
+		)
+	)
+	(wire
+		(pts
 			(xy 161.29 73.66) (xy 161.29 34.29)
 		)
@@
 	(wire
 		(pts
-			(xy 67.31 153.67) (xy 67.31 163.83)
+			(xy 69.85 153.67) (xy 69.85 170.18)
 		)
 		(stroke
@@
 	(wire
 		(pts
+			(xy 25.4 151.13) (xy 52.07 151.13)
+		)
+		(stroke
+			(width 0)
+			(type default)
+		)
+	)
+	(wire
+		(pts
+			(xy 52.07 170.18) (xy 69.85 170.18)
+		)
+		(stroke
+			(width 0)
+			(type default)
+		)
+	)
+	(wire
+		(pts
 			(xy 78.74 161.29) (xy 80.01 161.29)
 		)
@@
 	(wire
 		(pts
-			(xy 67.31 153.67) (xy 69.85 153.67)
-		)
-		(stroke
-			(width 0)
-			(type default)
-		)
-	)
-	(wire
-		(pts
 			(xy 114.3 121.92) (xy 114.3 111.76)
 		)
@@
 	(wire
 		(pts
-			(xy 109.22 158.75) (xy 109.22 186.69)
-		)
-		(stroke
-			(width 0)
-			(type default)
-		)
-	)
-	(wire
-		(pts
 			(xy 102.87 49.53) (xy 102.87 72.39)
 		)
@@
 	(wire
 		(pts
-			(xy 57.15 161.29) (xy 57.15 153.67)
-		)
-		(stroke
-			(width 0)
-			(type default)
-		)
-	)
-	(wire
-		(pts
 			(xy 114.3 111.76) (xy 124.46 111.76)
 		)
@@
 	(wire
 		(pts
-			(xy 116.84 163.83) (xy 67.31 163.83)
-		)
-		(stroke
-			(width 0)
-			(type default)
-		)
-	)
-	(wire
-		(pts
 			(xy 111.76 49.53) (xy 102.87 49.53)
 		)
@@
 	(wire
 		(pts
-			(xy 57.15 186.69) (xy 109.22 186.69)
-		)
-		(stroke
-			(width 0)
-			(type default)
-		)
-	)
-	(wire
-		(pts
-			(xy 57.15 153.67) (xy 67.31 153.67)
+			(xy 25.4 170.18) (xy 52.07 170.18)
+		)
+		(stroke
+			(width 0)
+			(type default)
+		)
+	)
+	(wire
+		(pts
+			(xy 25.4 160.02) (xy 25.4 170.18)
 		)
 		(stroke
@@
 	(wire
 		(pts
-			(xy 57.15 168.91) (xy 57.15 186.69)
-		)
-		(stroke
-			(width 0)
-			(type default)
-		)
-	)
-	(wire
-		(pts
 			(xy 73.66 115.57) (xy 87.63 115.57)
 		)
@@
 	(global_label "GND"
 		(shape bidirectional)
-		(at 78.74 161.29 180)
+		(at 78.74 161.29 270)
 		(fields_autoplaced yes)
 		(effects
@@
 	(global_label "RANGE_SELECT"
 		(shape bidirectional)
-		(at 116.84 153.67 90)
-		(fields_autoplaced yes)
-		(effects
-			(font
-				(size 1.27 1.27)
-			)
-			(justify left)
-		)
-		(property "Intersheetrefs" "${INTERSHEET_REFS}"
-			(at 116.84 135.7246 90)
+		(at 44.45 163.83 180)
+		(fields_autoplaced yes)
+		(effects
+			(font
+				(size 1.27 1.27)
+			)
+			(justify right)
+		)
+		(property "Intersheetrefs" "${INTERSHEET_REFS}"
+			(at 26.5046 163.83 0)
 			(show_name yes)
 			(effects
@@
 					(size 1.27 1.27)
 				)
-				(justify left)
+				(justify right)
 				(hide yes)
 			)
@@
 				(justify left)
 				(hide yes)
+			)
+		)
+	)
+	(symbol
+		(lib_id "Device:R")
+		(at 25.4 156.21 0)
+		(unit 1)
+		(exclude_from_sim no)
+		(in_bom yes)
+		(on_board yes)
+		(dnp no)
+		(fields_autoplaced yes)
+		(property "Reference" "R4"
+			(at 27.94 154.9399 0)
+			(effects
+				(font
+					(size 1.27 1.27)
+				)
+				(justify left)
+			)
+		)
+		(property "Value" "0.1 Ohm"
+			(at 27.94 157.4799 0)
+			(effects
+				(font
+					(size 1.27 1.27)
+				)
+				(justify left)
+			)
+		)
+		(property "Footprint" ""
+			(at 23.622 156.21 90)
+			(effects
+				(font
+					(size 1.27 1.27)
+				)
+				(hide yes)
+			)
+		)
+		(property "Datasheet" "~"
+			(at 25.4 156.21 0)
+			(effects
+				(font
+					(size 1.27 1.27)
+				)
+				(hide yes)
+			)
+		)
+		(property "Description" "Resistor"
+			(at 25.4 156.21 0)
+			(effects
+				(font
+					(size 1.27 1.27)
+				)
+				(hide yes)
+			)
+		)
+		(pin "1"
+		)
+		(pin "2"
+		)
+		(instances
+			(project ""
+				(path "/0cb921c9-5493-42a4-9366-73ecb4110608"
+					(reference "R4")
+					(unit 1)
+				)
 			)
 		)
@@
 	(symbol
 		(lib_id "Device:R")
-		(at 57.15 165.1 0)
+		(at 52.07 154.94 0)
 		(unit 1)
 		(exclude_from_sim no)
@@
 		(fields_autoplaced yes)
 		(property "Reference" "R2"
-			(at 59.69 163.8299 0)
-			(effects
-				(font
-					(size 1.27 1.27)
-				)
-				(justify left)
-			)
-		)
-		(property "Value" "R"
-			(at 59.69 166.3699 0)
+			(at 54.61 153.6699 0)
+			(effects
+				(font
+					(size 1.27 1.27)
+				)
+				(justify left)
+			)
+		)
+		(property "Value" "10 Ohm"
+			(at 54.61 156.2099 0)
 			(effects
 				(font
@@
 		)
 		(property "Footprint" ""
-			(at 55.372 165.1 90)
+			(at 50.292 154.94 90)
 			(effects
 				(font
@@
 		)
 		(property "Datasheet" "~"
-			(at 57.15 165.1 0)
+			(at 52.07 154.94 0)
 			(effects
 				(font
@@
 		)
 		(property "Description" "Resistor"
-			(at 57.15 165.1 0)
+			(at 52.07 154.94 0)
 			(effects
 				(font
@@
 	(symbol
 		(lib_id "Transistor_FET:BS170")
-		(at 114.3 158.75 0)
+		(at 49.53 163.83 0)
 		(unit 1)
 		(exclude_from_sim no)
@@
 		(fields_autoplaced yes)
 		(property "Reference" "Q1"
-			(at 120.65 157.4799 0)
+			(at 55.88 162.5599 0)
 			(effects
 				(font
@@
 		)
 		(property "Value" "BS170"
-			(at 120.65 160.0199 0)
+			(at 55.88 165.0999 0)
 			(effects
 				(font
@@
 		)
 		(property "Footprint" "Package_TO_SOT_THT:TO-92_Inline"
-			(at 119.38 160.655 0)
+			(at 54.61 165.735 0)
 			(effects
 				(font
@@
 		)
 		(property "Datasheet" "https://www.onsemi.com/pub/Collateral/BS170-D.PDF"
-			(at 119.38 162.56 0)
+			(at 54.61 167.64 0)
 			(effects
 				(font
@@
 		)
 		(property "Description" "0.5A Id, 60V Vds, N-Channel MOSFET, TO-92"
-			(at 114.3 158.75 0)
-			(effects
-				(font
+			(at 49.53 163.83 0)
+			(effects
+				(font

Commit message: Updated few in ur sch
Parts:
- added J2: TEST_SOCKET, symbol Connector:Screw_Terminal_01x03
- C1: value C -> 0.1uF
- R1: value R -> 1M Ohm
- R3: value R -> 10k Ohm
Connections:
- net CURRENT_IN: now also J2.2 (Pin_2)
- net GND: now also J2.3 (Pin_3)
- new net V_SWEEP: J2.1 (Pin_1)
Changed lines of the file:
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@@
+		)
+	)
+	(global_label "V_SWEEP"
+		(shape bidirectional)
+		(at 127 152.4 180)
+		(fields_autoplaced yes)
+		(effects
+			(font
+				(size 1.27 1.27)
+			)
+			(justify right)
+		)
+		(property "Intersheetrefs" "${INTERSHEET_REFS}"
+			(at 114.6184 152.4 0)
+			(effects
+				(font
+					(size 1.27 1.27)
+				)
+				(justify right)
+				(hide yes)
+			)
 		)
 	)
@@
 				)
 				(justify left)
+				(hide yes)
+			)
+		)
+	)
+	(global_label "CURRENT_IN"
+		(shape bidirectional)
+		(at 127 154.94 180)
+		(fields_autoplaced yes)
+		(effects
+			(font
+				(size 1.27 1.27)
+			)
+			(justify right)
+		)
+		(property "Intersheetrefs" "${INTERSHEET_REFS}"
+			(at 111.413 154.94 0)
+			(effects
+				(font
+					(size 1.27 1.27)
+				)
+				(justify right)
 				(hide yes)
 			)
@@
 	)
 	(symbol
+		(lib_id "Connector:Screw_Terminal_01x03")
+		(at 132.08 154.94 0)
+		(unit 1)
+		(exclude_from_sim no)
+		(in_bom yes)
+		(on_board yes)
+		(dnp no)
+		(fields_autoplaced yes)
+		(property "Reference" "J2"
+			(at 134.62 153.6699 0)
+			(effects
+				(font
+					(size 1.27 1.27)
+				)
+				(justify left)
+			)
+		)
+		(property "Value" "TEST_SOCKET"
+			(at 134.62 156.2099 0)
+			(effects
+				(font
+					(size 1.27 1.27)
+				)
+				(justify left)
+			)
+		)
+		(property "Footprint" ""
+			(at 132.08 154.94 0)
+			(effects
+				(font
+					(size 1.27 1.27)
+				)
+				(hide yes)
+			)
+		)
+		(property "Datasheet" "~"
+			(at 132.08 154.94 0)
+			(effects
+				(font
+					(size 1.27 1.27)
+				)
+				(hide yes)
+			)
+		)
+		(property "Description" "Generic screw terminal, single row, 01x03, script generated (kicad-library-utils/schlib/autogen/connector/)"
+			(at 132.08 154.94 0)
+			(effects
+				(font
+					(size 1.27 1.27)
+				)
+				(hide yes)
+			)
+		)
+		(pin "1"
+		)
+		(pin "2"
+		)
+		(pin "3"
+		)
+		(instances
+			(project ""
+				(path "/0cb921c9-5493-42a4-9366-73ecb4110608"
+					(reference "J2")
+					(unit 1)
+				)
+			)
+		)
+	)
+	(symbol
+		(lib_id "power:GND")
+		(at 127 157.48 0)
+		(unit 1)
+		(exclude_from_sim no)
+		(in_bom yes)
+		(on_board yes)
+		(dnp no)
+		(fields_autoplaced yes)
+		(property "Reference" "#PWR01"
+			(at 127 163.83 0)
+			(effects
+				(font
+					(size 1.27 1.27)
+				)
+				(hide yes)
+			)
+		)
+		(property "Value" "GND"
+			(at 127 162.56 0)
+			(effects
+				(font
+					(size 1.27 1.27)
+				)
+			)
+		)
+		(property "Footprint" ""
+			(at 127 157.48 0)
+			(effects
+				(font
+					(size 1.27 1.27)
+				)
+				(hide yes)
+			)
+		)
+		(property "Datasheet" ""
+			(at 127 157.48 0)
+			(effects
+				(font
+					(size 1.27 1.27)
+				)
+				(hide yes)
+			)
+		)
+		(property "Description" "Power symbol creates a global label with name \"GND\" , ground"
+			(at 127 157.48 0)
+			(effects
+				(font
+					(size 1.27 1.27)
+				)
+				(hide yes)
+			)
+		)
+		(pin "1"
+		)
+		(instances
+			(project ""
+				(path "/0cb921c9-5493-42a4-9366-73ecb4110608"
+					(reference "#PWR01")
+					(unit 1)
+				)
+			)
+		)
+	)
+	(symbol
 		(lib_id "Amplifier_Operational:TL072")
 		(at 119.38 99.06 0)
@@
 			)
 		)
-		(property "Value" "R"
+		(property "Value" "10k Ohm"
 			(at 127 119.3799 0)
 			(effects
@@
 		(on_board yes)
 		(dnp no)
-		(fields_autoplaced yes)
 		(property "Reference" "R1"
 			(at 95.25 110.4899 0)
@@
 			)
 		)
-		(property "Value" "R"
+		(property "Value" "1M Ohm"
 			(at 95.25 113.0299 0)
 			(effects
@@
 			)
 		)
-		(property "Value" "C"
+		(property "Value" "0.1uF"
 			(at 96.52 81.2799 0)
 			(effects
