File: Auralab_Workstation/rp2040_core.kicad_sch (KiCad schematic)
At the start: 20 parts, among them Q1 BC847, U1 RP2040, U2 W25Q128JVS, Y1 Crystal_GND24

Commit message: Now updated..
Parts:
- added C5: 100nF, symbol Device:C
- added R7: 1k, symbol Device:R
Connections:
- net ADC_MISO: now also U1.5 (GPIO3); no longer U1.7 (GPIO5)
- net ADC_SCLK: now also U1.4 (GPIO2); no longer U1.6 (GPIO4)
- net GND: now also C5.2
- net I2C_SCL: now also U1.7 (GPIO5); no longer U1.5 (GPIO3)
- net I2C_SDA: now also U1.6 (GPIO4); no longer U1.4 (GPIO2)
- net SWEEP_PWM: now reaches U1.13 (GPIO10)
- net SWEEP_PWM: now also R7.1
- new net: C5.1, R7.2
- no-connect marks 17 -> 16
Other:
- moved on the sheet: D2, R6

Commit message: Made few changes in IN2A66 in urs
Parts:
- added SW1: RotaryEncoder_Switch, symbol Device:RotaryEncoder_Switch
Connections:
- net GND: now also SW1.C, SW1.S2
- net ROT_B: now reaches U1.14 (GPIO11)
- net ROT_B: now also SW1.B
- net BTN_MENU_NEXT renamed ROT_A
- net ROT_A: now also SW1.A
- net BTN_MENU_SELECT renamed ROT_SW
- net ROT_SW: now also SW1.S1
- no-connect marks 16 -> 15

Commit message: Updated footprints for rp2040
Parts:
- BZ1: footprint (none) -> Buzzer_Beeper:Buzzer_CUI_CPT-9019S-SMT
- C1, C2, C3, C4, C5: footprint (none) -> Capacitor_SMD:C_0805_2012Metric_Pad1.18x1.45mm_HandSolder
- Clean_Analog_Filter1: renamed from Clean_Analog_Filter; footprint (none) -> Capacitor_SMD:C_0805_2012Metric_Pad1.18x1.45mm_HandSolder
- D1, D2: footprint (none) -> LED_SMD:LED_0805_2012Metric_Pad1.15x1.40mm_HandSolder
- Digital_Filter1: renamed from Digital_Filter; footprint (none) -> Capacitor_SMD:C_0805_2012Metric_Pad1.18x1.45mm_HandSolder
- R1, R2, R3, R4, R5, R6, R7: footprint (none) -> Resistor_SMD:R_0805_2012Metric_Pad1.20x1.40mm_HandSolder
- Regulator_Filter1: renamed from Regulator_Filter; footprint (none) -> Capacitor_SMD:C_0805_2012Metric_Pad1.18x1.45mm_HandSolder
- SW1: footprint (none) -> Rotary_Encoder:RotaryEncoder_Alps_EC11E-Switch_Vertical_H20mm
- Y1: footprint (none) -> Crystal:Crystal_SMD_3225-4Pin_3.2x2.5mm_HandSoldering
Changed lines of the file:
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@@
 			)
 		)
-		(property "Footprint" ""
+		(property "Footprint" "Crystal:Crystal_SMD_3225-4Pin_3.2x2.5mm_HandSoldering"
 			(at 196.85 46.99 0)
 			(effects
@@
 			)
 		)
-		(property "Footprint" ""
+		(property "Footprint" "Capacitor_SMD:C_0805_2012Metric_Pad1.18x1.45mm_HandSolder"
 			(at 204.1652 33.02 0)
 			(effects
@@
 			)
 		)
-		(property "Footprint" ""
+		(property "Footprint" "Resistor_SMD:R_0805_2012Metric_Pad1.20x1.40mm_HandSolder"
 			(at 212.09 67.818 90)
 			(effects
@@
 			)
 		)
-		(property "Footprint" ""
+		(property "Footprint" "Capacitor_SMD:C_0805_2012Metric_Pad1.18x1.45mm_HandSolder"
 			(at 216.8652 73.66 0)
 			(effects
@@
 		(dnp no)
 		(fields_autoplaced yes)
-		(property "Reference" "Clean_Analog_Filter"
+		(property "Reference" "Clean_Analog_Filter1"
 			(at 156.21 30.4799 0)
 			(effects
@@
 			)
 		)
-		(property "Footprint" ""
+		(property "Footprint" "Capacitor_SMD:C_0805_2012Metric_Pad1.18x1.45mm_HandSolder"
 			(at 153.3652 35.56 0)
 			(effects
@@
 			(project "rp2040_core"
 				(path "/7b3e6f41-6595-497a-a0ba-4d530102dce3"
-					(reference "Clean_Analog_Filter")
+					(reference "Clean_Analog_Filter1")
 					(unit 1)
 				)
@@
 			)
 		)
-		(property "Footprint" ""
+		(property "Footprint" "Resistor_SMD:R_0805_2012Metric_Pad1.20x1.40mm_HandSolder"
 			(at 57.15 76.708 90)
 			(effects
@@
 			)
 		)
-		(property "Footprint" ""
+		(property "Footprint" "Capacitor_SMD:C_0805_2012Metric_Pad1.18x1.45mm_HandSolder"
 			(at 186.3852 33.02 0)
 			(effects
@@
 			)
 		)
-		(property "Footprint" ""
+		(property "Footprint" "Rotary_Encoder:RotaryEncoder_Alps_EC11E-Switch_Vertical_H20mm"
 			(at 46.99 149.606 0)
 			(effects
@@
 			)
 		)
-		(property "Footprint" ""
+		(property "Footprint" "Resistor_SMD:R_0805_2012Metric_Pad1.20x1.40mm_HandSolder"
 			(at 49.53 116.078 90)
 			(effects
@@
 			)
 		)
-		(property "Footprint" ""
+		(property "Footprint" "Resistor_SMD:R_0805_2012Metric_Pad1.20x1.40mm_HandSolder"
 			(at 74.422 31.75 90)
 			(effects
@@
 			)
 		)
-		(property "Footprint" ""
+		(property "Footprint" "Resistor_SMD:R_0805_2012Metric_Pad1.20x1.40mm_HandSolder"
 			(at 161.29 50.038 90)
 			(effects
@@
 			)
 		)
-		(property "Footprint" ""
+		(property "Footprint" "Resistor_SMD:R_0805_2012Metric_Pad1.20x1.40mm_HandSolder"
 			(at 186.69 99.568 90)
 			(effects
@@
 			)
 		)
-		(property "Footprint" ""
+		(property "Footprint" "LED_SMD:LED_0805_2012Metric_Pad1.15x1.40mm_HandSolder"
 			(at 168.91 48.26 0)
 			(effects
@@
 			)
 		)
-		(property "Footprint" ""
+		(property "Footprint" "Resistor_SMD:R_0805_2012Metric_Pad1.20x1.40mm_HandSolder"
 			(at 57.15 70.358 90)
 			(effects
@@
 		(on_board yes)
 		(dnp no)
-		(property "Reference" "Regulator_Filter"
+		(property "Reference" "Regulator_Filter1"
 			(at 133.35 30.4799 0)
 			(effects
@@
 			)
 		)
-		(property "Footprint" ""
+		(property "Footprint" "Capacitor_SMD:C_0805_2012Metric_Pad1.18x1.45mm_HandSolder"
 			(at 130.5052 35.56 0)
 			(effects
@@
 			(project "rp2040_core"
 				(path "/7b3e6f41-6595-497a-a0ba-4d530102dce3"
-					(reference "Regulator_Filter")
+					(reference "Regulator_Filter1")
 					(unit 1)
 				)
@@
 			)
 		)
-		(property "Footprint" ""
+		(property "Footprint" "LED_SMD:LED_0805_2012Metric_Pad1.15x1.40mm_HandSolder"
 			(at 194.31 97.79 0)
 			(effects
@@
 			)
 		)
-		(property "Footprint" ""
+		(property "Footprint" "Capacitor_SMD:C_0805_2012Metric_Pad1.18x1.45mm_HandSolder"
 			(at 243.5352 102.87 0)
 			(effects
@@
 		(dnp no)
 		(fields_autoplaced yes)
-		(property "Reference" "Digital_Filter"
+		(property "Reference" "Digital_Filter1"
 			(at 111.76 30.4799 0)
 			(effects
@@
 			)
 		)
-		(property "Footprint" ""
+		(property "Footprint" "Capacitor_SMD:C_0805_2012Metric_Pad1.18x1.45mm_HandSolder"
 			(at 108.9152 35.56 0)
 			(effects
@@
 			(project ""
 				(path "/7b3e6f41-6595-497a-a0ba-4d530102dce3"
-					(reference "Digital_Filter")
+					(reference "Digital_Filter1")
 					(unit 1)
 				)
@@
 			)
 		)
-		(property "Footprint" ""
+		(property "Footprint" "Capacitor_SMD:C_0805_2012Metric_Pad1.18x1.45mm_HandSolder"
 			(at 92.4052 35.56 0)
 			(effects
@@
 			)
 		)
-		(property "Footprint" ""
+		(property "Footprint" "Buzzer_Beeper:Buzzer_CUI_CPT-9019S-SMT"
 			(at 62.865 104.14 90)
 			(effects

Commit message: Power management le few changes made inum full ah complete panle..
Parts:
- added J1: Conn_01x14_Socket, Connector_PinSocket_2.54mm:PinSocket_1x14_P2.54mm_Vertical, symbol Connector:Conn_01x14_Socket
- added R8: 100 Ohm, Resistor_SMD:R_0805_2012Metric_Pad1.20x1.40mm_HandSolder, symbol Device:R
Connections:
- net +3.3V: now also J1.1 (Pin_1)
- net GND: now also J1.2 (Pin_2)
- net TFT_CS: now also J1.3 (Pin_3)
- net TFT_DC: now also J1.5 (Pin_5)
- net TFT_MOSI: now also J1.6 (Pin_6)
- net TFT_RST: now also J1.4 (Pin_4)
- net TFT_SCLK: now also J1.7 (Pin_7)
- net USB_DM: no longer U1.46 (USB_DM)
- net USB_DP: no longer U1.47 (USB_DP)
- net USB_D_M: now also U1.46 (USB_DM)
- net USB_D_P: now also U1.47 (USB_DP)
- new net: J1.8 (Pin_8), R8.2
- new net +5V: R8.1
- no-connect marks 15 -> 21

Commit message: Power management connections checked its perfect now
Connections:
- net POT_SPI_CS: now reaches U1.15 (GPIO12)
- net POT_SPI_SCK: now reaches U1.16 (GPIO13)
- net POT_SPI_MOSI: now reaches U1.17 (GPIO14)
- no-connect marks 21 -> 18
Other:
- moved on the sheet: D2, R6
Changed lines of the file:
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@@
 	)
 	(no_connect
-		(at 154.94 99.06)
-	)
-	(no_connect
 		(at 154.94 66.04)
 	)
 	(no_connect
-		(at 154.94 96.52)
-	)
-	(no_connect
 		(at 257.81 49.53)
 	)
@@
 	)
 	(no_connect
-		(at 154.94 101.6)
-	)
-	(no_connect
 		(at 257.81 44.45)
 	)
@@
 	(wire
 		(pts
+			(xy 154.94 99.06) (xy 171.45 99.06)
+		)
+		(stroke
+			(width 0)
+			(type default)
+		)
+	)
+	(wire
+		(pts
 			(xy 209.55 52.07) (xy 196.85 52.07)
 		)
@@
 		)
 	)
+	(global_label "POT_SPI_MOSI"
+		(shape output)
+		(at 154.94 101.6 0)
+		(fields_autoplaced yes)
+		(effects
+			(font
+				(size 1.27 1.27)
+			)
+			(justify left)
+		)
+		(property "Intersheetrefs" "${INTERSHEET_REFS}"
+			(at 171.109 101.6 0)
+			(effects
+				(font
+					(size 1.27 1.27)
+				)
+				(justify left)
+				(hide yes)
+			)
+		)
+	)
 	(global_label "TFT_MOSI"
 		(shape bidirectional)
@@
 		)
 	)
+	(global_label "POT_SPI_CS"
+		(shape output)
+		(at 154.94 96.52 0)
+		(fields_autoplaced yes)
+		(effects
+			(font
+				(size 1.27 1.27)
+			)
+			(justify left)
+		)
+		(property "Intersheetrefs" "${INTERSHEET_REFS}"
+			(at 168.9923 96.52 0)
+			(effects
+				(font
+					(size 1.27 1.27)
+				)
+				(justify left)
+				(hide yes)
+			)
+		)
+	)
 	(global_label "XOUT"
 		(shape output)
@@
 	(global_label "ALERT_LED"
 		(shape bidirectional)
-		(at 198.12 97.79 0)
+		(at 217.17 86.36 0)
 		(fields_autoplaced yes)
 		(effects
@@
 		)
 		(property "Intersheetrefs" "${INTERSHEET_REFS}"
-			(at 212.1345 97.79 0)
+			(at 231.1845 86.36 0)
 			(effects
 				(font
@@
 		)
 	)
+	(global_label "POT_SPI_SCK"
+		(shape output)
+		(at 171.45 99.06 0)
+		(fields_autoplaced yes)
+		(effects
+			(font
+				(size 1.27 1.27)
+			)
+			(justify left)
+		)
+		(property "Intersheetrefs" "${INTERSHEET_REFS}"
+			(at 186.7723 99.06 0)
+			(effects
+				(font
+					(size 1.27 1.27)
+				)
+				(justify left)
+				(hide yes)
+			)
+		)
+	)
 	(global_label "XOUT"
 		(shape output)
@@
 	(symbol
 		(lib_id "power:GND")
-		(at 182.88 97.79 0)
+		(at 201.93 86.36 0)
 		(unit 1)
 		(exclude_from_sim no)
@@
 		(dnp no)
 		(property "Reference" "#PWR022"
-			(at 182.88 104.14 0)
+			(at 201.93 92.71 0)
 			(effects
 				(font
@@
 		)
 		(property "Value" "GND"
-			(at 180.848 98.298 0)
+			(at 199.898 86.868 0)
 			(effects
 				(font
@@
 		)
 		(property "Footprint" ""
-			(at 182.88 97.79 0)
+			(at 201.93 86.36 0)
 			(effects
 				(font
@@
 		)
 		(property "Datasheet" ""
-			(at 182.88 97.79 0)
+			(at 201.93 86.36 0)
 			(effects
 				(font
@@
 		)
 		(property "Description" "Power symbol creates a global label with name \"GND\" , ground"
-			(at 182.88 97.79 0)
+			(at 201.93 86.36 0)
 			(effects
 				(font
@@
 	(symbol
 		(lib_id "Device:R")
-		(at 186.69 97.79 90)
+		(at 205.74 86.36 90)
 		(unit 1)
 		(exclude_from_sim no)
@@
 		(dnp no)
 		(property "Reference" "R6"
-			(at 186.69 97.79 90)
+			(at 205.74 86.36 90)
 			(effects
 				(font
@@
 		)
 		(property "Value" "220 Ohm"
-			(at 186.69 95.758 90)
+			(at 205.74 84.328 90)
 			(effects
 				(font
@@
 		)
 		(property "Footprint" "Resistor_SMD:R_0805_2012Metric_Pad1.20x1.40mm_HandSolder"
-			(at 186.69 99.568 90)
+			(at 205.74 88.138 90)
 			(effects
 				(font
@@
 		)
 		(property "Datasheet" "~"
-			(at 186.69 97.79 0)
+			(at 205.74 86.36 0)
 			(effects
 				(font
@@
 		)
 		(property "Description" "Resistor"
-			(at 186.69 97.79 0)
+			(at 205.74 86.36 0)
 			(effects
 				(font
@@
 	(symbol
 		(lib_id "Device:LED")
-		(at 194.31 97.79 0)
+		(at 213.36 86.36 0)
 		(unit 1)
 		(exclude_from_sim no)
@@
 		(dnp no)
 		(property "Reference" "D2"
-			(at 194.818 95.758 0)
+			(at 213.868 84.328 0)
 			(effects
 				(font
@@
 		)
 		(property "Value" "LED"
-			(at 195.072 100.076 0)
+			(at 214.122 88.646 0)
 			(effects
 				(font
@@
 		)
 		(property "Footprint" "LED_SMD:LED_0805_2012Metric_Pad1.15x1.40mm_HandSolder"
-			(at 194.31 97.79 0)
+			(at 213.36 86.36 0)
 			(effects
 				(font
@@
 		)
 		(property "Datasheet" "~"
-			(at 194.31 97.79 0)
+			(at 213.36 86.36 0)
 			(effects
 				(font
@@
 		)
 		(property "Description" "Light emitting diode"
-			(at 194.31 97.79 0)
+			(at 213.36 86.36 0)
 			(effects
 				(font
@@
 		)
 		(property "Sim.Pins" "1=K 2=A"
-			(at 194.31 97.79 0)
+			(at 213.36 86.36 0)
 			(effects
 				(font

Commit message: Check analog part
Connections:
- net V_filtered: now reaches C5.1, R7.2
Changed lines of the file:
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@@
 	(paper "A4")
+	(junction
+		(at 215.9 66.04)
+		(diameter 0)
+		(color 0 0 0 0)
+	)
 	(junction
 		(at 33.02 153.67)
@@
 		)
 	)
+	(wire
+		(pts
+			(xy 220.98 66.04) (xy 215.9 66.04)
+		)
+		(stroke
+			(width 0)
+			(type default)
+		)
+	)
 	(global_label "USB_D_M"
 		(shape bidirectional)
@@
 				(hide yes)
 			)
+		)
+	)
+	(global_label "V_filtered"
+		(shape bidirectional)
+		(at 220.98 66.04 0)
+		(fields_autoplaced yes)
+		(effects
+			(font
+				(size 1.27 1.27)
+			)
+			(justify left)
+		)
+		(property "Intersheetrefs" "${INTERSHEET_REFS}"
+			(at 233.9665 66.04 0)
+			(effects
+				(font
+					(size 1.27 1.27)
+				)
+				(justify left)
+				(hide yes)
+			)

Commit message: Check ERC
Parts:
- added J2: Conn_01x03, Connector_PinHeader_2.54mm:PinHeader_1x03_P2.54mm_Vertical, symbol Connector_Generic:Conn_01x03
- added R9: 10k Ohm, Resistor_SMD:R_0805_2012Metric_Pad1.20x1.40mm_HandSolder, symbol Device:R
- added SW2: SW_Push, Button_Switch_THT:SW_PUSH-12mm_Wuerth-430476085716, symbol Switch:SW_Push
- D1: value LED -> POWER_ON_LED
Connections:
- net GND: now also J2.3 (Pin_3), SW2.2
- net TFT_MISO: now reaches U1.18 (GPIO15)
- net TFT_MISO: now also J1.9 (Pin_9)
- net SWCLK: now reaches U1.24 (SWCLK)
- net SWCLK: now also J2.1 (Pin_1)
- net SWD: now reaches U1.25 (SWD)
- net SWD: now also J2.2 (Pin_2)
- net +3.3V renamed +3V3_DIGITAL
- net +3V3_DIGITAL: now also R9.1; no longer U1.26 (RUN)
- net +5V renamed +5V_RAW
- net ADC_3V3 renamed +3V3_ANALOG
- new net: R9.2, SW2.1, U1.26 (RUN)
- no-connect marks 18 -> 14
Other:
- moved on the sheet: BZ1, C1, C2, C3, C4, C5, Clean_Analog_Filter1, D1, D2, Digital_Filter1, J1, Q1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

Commit message: ERC checked
Parts:
- renumbered C3 to C10, C4 to C11, C5 to C12, C1 to C8, C2 to C9, D1 to D8, D2 to D9, J2 to J6, J1 to J7, Q1 to Q2, R4 to R15, R6 to R16, R5 to R17, R2 to R18, R3 to R19, R1 to R20, R9 to R21, R8 to R22, R7 to R23, SW1 to SW2, SW2 to SW3, U1 to U10, U2 to U11
