File: Auralab_Workstation/AuralabWorkstation_1.kicad_pcb (KiCad board)
At the start: 6 copper layers, 128.6 x 96.9 mm, 80 parts, among them J1 Conn_Coaxial, J2 TEST_SOCKET, J3 USB_C_Receptacle_USB2.0_16P, J4 Screw_Terminal_01x03, J5 Conn_01x02_Socket, J6 Conn_01x03, J7 Conn_01x14_Socket, M1 MountingHole_3mm_Pad_TopBottom, M2 MountingHole_3mm_Pad_TopBottom, M3 MountingHole_3mm_Pad_TopBottom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

Commit message: Add files via upload
Parts:
- moved C2 0.80 mm to (38.0, 69.0)
Routing:
- net GND: track 0.00 -> 389.2 mm, vias 0 -> 6
- net GNDA: track 0.00 -> 227.0 mm, vias 0 -> 7
- net +3V3_DIGITAL: track 142.9 -> 226.1 mm, vias 0 -> 3
- net POT_SPI_MOSI: track 0.00 -> 76.4 mm, vias 0 -> 2
- net +Vout: track 45.1 -> 118.9 mm, vias 0 -> 3
- net V_filtered: track 2.50 -> 66.8 mm, vias 0 -> 2
- net ROT_B: track 0.00 -> 59.6 mm
- net POT_SPI_CS: track 0.00 -> 50.5 mm, vias 0 -> 2
- net -Vout: track 60.0 -> 110.0 mm, vias 1 -> 4
- net TFT_MOSI: track 0.00 -> 34.9 mm
- net TFT_RST: track 0.00 -> 28.0 mm, vias 0 -> 2
- net TFT_CS: track 0.00 -> 27.7 mm, vias 0 -> 3
- net +5V_RAW: track 64.2 -> 83.7 mm, vias 1 -> 2
- net /FBP: track 23.1 -> 41.4 mm, vias 1 -> 3
- net A7: track 41.4 -> 23.3 mm, vias 1 -> 2
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
Commit message: ..
Parts:
- moved U11 93.9 mm to (141.4, 68.5), turned to 90 degrees
- moved U9 56.1 mm to (139.9, 52.5)
- moved BZ1 44.5 mm to (140.5, 82.9)
- moved C8 43.0 mm to (128.7, 72.1)
- moved Y1 40.6 mm to (121.1, 72.2)
- moved L1 38.5 mm to (75.8, 50.0)
- moved C7 37.6 mm to (112.2, 72.4)
- moved R11 35.9 mm to (64.1, 72.7)
- moved U5 34.9 mm to (112.4, 58.6), turned to 180 degrees
- moved D4 33.3 mm to (72.8, 72.2)
- moved R12 26.8 mm to (60.3, 67.1)
- moved CleanAnalogFilter 26.3 mm to (113.9, 46.0)
- moved U8 22.2 mm to (89.5, 62.8)
- moved D5 21.7 mm to (71.0, 65.6)
- moved SW3 20.7 mm to (85.3, 24.5)
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Routing:
- net GND: track 389.2 -> 0.00 mm, vias 6 -> 0
- net GNDA: track 227.0 -> 0.00 mm, vias 7 -> 0
- net +3V3_DIGITAL: track 226.1 -> 0.00 mm, vias 3 -> 0
- net +Vout: track 118.9 -> 0.00 mm, vias 3 -> 0
- net -Vout: track 110.0 -> 0.00 mm, vias 4 -> 0
- net +5V_RAW: track 83.7 -> 0.00 mm, vias 2 -> 0
- net POT_SPI_MOSI: track 76.4 -> 0.00 mm, vias 2 -> 0
- net VBUS_SYSTEM: track 71.3 -> 0.00 mm, vias 2 -> 0
- net V_filtered: track 66.8 -> 0.00 mm, vias 2 -> 0
- net ROT_B: track 59.6 -> 0.00 mm
- net Net-(J7-Pin_8): track 56.2 -> 0.00 mm, vias 1 -> 0
- net POT_SPI_CS: track 50.5 -> 0.00 mm, vias 2 -> 0
- net /FBP: track 41.4 -> 0.00 mm, vias 3 -> 0
- net CURRENT_IN: track 37.5 -> 0.00 mm, vias 1 -> 0
- net TFT_MOSI: track 34.9 -> 0.00 mm
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