File: Auralab_Workstation/maincontestpcb_vishal.kicad_pcb (KiCad board)
At the start: 6 copper layers, 128.6 x 96.9 mm, 80 parts, among them J1 Conn_Coaxial, J2 TEST_SOCKET, J3 USB_C_Receptacle_USB2.0_16P, J4 Screw_Terminal_01x03, J5 Conn_01x02_Socket, J6 Conn_01x03, J7 Conn_01x14_Socket, M1 MountingHole_3mm_Pad_TopBottom, M2 MountingHole_3mm_Pad_TopBottom, M3 MountingHole_3mm_Pad_TopBottom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

Commit message: ..
Parts:
- moved D4 93.1 mm to (15.0, 22.0)
- moved U5 78.3 mm to (28.0, 38.0)
- moved U11 77.2 mm to (118.0, 38.0), turned to 0 degrees
- moved C11 52.3 mm to (118.0, 32.0), turned to 0 degrees
- moved C6 44.6 mm to (57.0, 24.0), turned to 180 degrees
- moved C5 39.5 mm to (43.0, 24.0), turned to 180 degrees
- moved F1 39.0 mm to (25.0, 22.0), turned to 180 degrees
- moved J1 38.3 mm to (18.0, 82.0), turned to 180 degrees
- moved U1 36.5 mm to (53.0, 82.0)
- moved J7 35.2 mm to (118.0, 72.0), turned to 180 degrees
- moved FB1 33.4 mm to (32.0, 22.0), turned to 0 degrees
- moved U10 32.7 mm to (80.0, 48.0)
- moved J2 31.8 mm to (98.0, 78.0), turned to 180 degrees
- moved SW1 30.1 mm to (38.0, 72.0), turned to 0 degrees
- moved C3 29.3 mm to (20.0, 38.0), turned to 180 degrees
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Routing:
- net +3V3_DIGITAL: track 142.9 -> 0.00 mm
- net VBUS_SYSTEM: track 68.0 -> 0.00 mm, vias 1 -> 0
- net +5V_RAW: track 64.2 -> 0.00 mm, vias 1 -> 0
- net -Vout: track 60.0 -> 0.00 mm, vias 1 -> 0
- net Net-(J7-Pin_8): track 58.5 -> 0.00 mm
- net +Vout: track 45.1 -> 0.00 mm
- net A7: track 41.4 -> 0.00 mm, vias 1 -> 0
- net CURRENT_IN: track 38.4 -> 0.00 mm
- net /+IN_ADC: track 33.8 -> 0.00 mm
- net A6: track 28.8 -> 0.00 mm, vias 1 -> 0
- net /Non-inv Input OpAmp: track 28.6 -> 0.00 mm
- net Net-(D8-K): track 25.7 -> 0.00 mm, vias 1 -> 0
- net Net-(U1B--): track 25.1 -> 0.00 mm
- net Net-(D7-K): track 25.1 -> 0.00 mm, vias 1 -> 0
- net /FBP: track 23.1 -> 0.00 mm, vias 1 -> 0
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Other:
- board outline removed
