File: Auralab_Workstation/maincontest.kicad_pcb (KiCad board)
At the start: 6 copper layers, 80 x 68.5 mm, 76 parts, among them J1 Conn_Coaxial, J2 TEST_SOCKET, J3 USB_C_Receptacle_USB2.0_16P, J4 Screw_Terminal_01x03, J5 Conn_01x02_Socket, J6 Conn_01x03, J7 Conn_01x14_Socket, Q1 BS170, Q2 BC847, SW1 SW_SPDT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

Commit message: pcb..
Parts:
- added M1: MountingHole_3mm_Pad_TopBottom, MountingHole:MountingHole_3mm_Pad_TopBottom, F.Cu at (25.3, 25.4)
- added M2: MountingHole_3mm_Pad_TopBottom, MountingHole:MountingHole_3mm_Pad_TopBottom, F.Cu at (135.0, 27.2)
- added M3: MountingHole_3mm_Pad_TopBottom, MountingHole:MountingHole_3mm_Pad_TopBottom, F.Cu at (24.8, 134.3)
- added M4: MountingHole_3mm_Pad_TopBottom, MountingHole:MountingHole_3mm_Pad_TopBottom, F.Cu at (135.5, 133.9)
- moved R12 200.1 mm to (243.5, 119.7)
- moved SW3 190.0 mm to (253.2, 77.8)
- moved L2 176.0 mm to (245.6, 131.9)
- moved U1 168.5 mm to (204.9, 139.6), turned to 180 degrees
- moved J2 168.3 mm to (243.1, 96.2)
- moved U8 167.2 mm to (247.9, 67.4)
- moved L1 164.4 mm to (230.0, 134.5)
- moved D5 159.2 mm to (243.8, 112.5)
- moved D4 157.9 mm to (243.0, 106.9)
- moved U2 154.6 mm to (192.8, 139.1)
- moved R19 154.6 mm to (210.8, 89.6)
- moved R22 152.4 mm to (208.0, 94.8)
- moved Q1 151.1 mm to (228.3, 75.7)
- moved D9 150.7 mm to (229.0, 126.3)
- moved BZ1 150.4 mm to (220.1, 67.6)
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Other:
- board size 80 x 68.5 mm -> 120 x 120 mm

Commit message: Add files via upload
Parts:
- removed M1, M2, M3, M4: MountingHole_3mm_Pad_TopBottom, MountingHole:MountingHole_3mm_Pad_TopBottom
- moved J4 217.9 mm to (228.0, 121.0), turned to 0 degrees
- moved D5 192.0 mm to (52.0, 104.0)
- moved D4 191.3 mm to (62.0, 45.0)
- moved D7 172.2 mm to (150.0, 149.0), turned to 90 degrees
- moved L1 157.6 mm to (80.0, 86.0), turned to 90 degrees
- moved L2 152.7 mm to (100.0, 86.0), turned to 90 degrees
- moved D3 150.5 mm to (78.0, 114.0)
- moved R15 139.9 mm to (62.0, 55.0), turned to 90 degrees
- moved R9 138.1 mm to (100.0, 149.0), turned to 90 degrees
- moved R11 137.7 mm to (62.0, 112.0), turned to 90 degrees
- moved SW3 135.8 mm to (125.0, 33.0)
- moved BZ1 129.0 mm to (120.0, 149.0)
- moved C6 123.8 mm to (94.0, 56.0)
- moved U8 122.9 mm to (125.0, 65.0)
- moved U6 122.0 mm to (52.0, 50.0), turned to 90 degrees
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Routing:
- net GND: track 0.00 -> 717.6 mm, vias 0 -> 14
- net +3V3_DIGITAL: track 0.00 -> 483.5 mm, vias 0 -> 10
- net GNDA: track 0.00 -> 391.1 mm, vias 0 -> 4
- net Net-(J7-Pin_8): track 0.00 -> 381.5 mm, vias 0 -> 1
- net +5V_RAW: track 0.00 -> 316.3 mm, vias 0 -> 5
- net RANGE_SELECT: track 0.00 -> 282.6 mm, vias 0 -> 3
- net ROT_A: track 0.00 -> 275.6 mm, vias 0 -> 1
- net +Vout: track 0.00 -> 214.7 mm, vias 0 -> 5
- net -Vout: track 0.00 -> 212.0 mm, vias 0 -> 3
- net ALERT_LED: track 0.00 -> 199.4 mm, vias 0 -> 2
- net Net-(D2-A): track 0.00 -> 174.5 mm, vias 0 -> 3
- net Net-(J3-CC2): track 0.00 -> 173.1 mm, vias 0 -> 2
- net Net-(J3-CC1): track 0.00 -> 173.1 mm, vias 0 -> 2
- net VBUS_SYSTEM: track 0.00 -> 172.7 mm, vias 0 -> 5
- net /+IN_ADC: track 0.00 -> 171.6 mm, vias 0 -> 3
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Other:
- board size 120 x 120 mm -> 246 x 141 mm

Commit message: Add files via upload
Parts:
- Regulator_Filter1: moved to B.Cu
- moved R17 23.1 mm to (159.0, 26.0), turned to 180 degrees
- turned Regulator_Filter1 to 180 degrees
Routing:
- net +1.1V: track 0.00 -> 105.1 mm, vias 0 -> 5
- net ADC_CS: track 0.00 -> 101.5 mm, vias 0 -> 1
- net BUZZER_CTRL: track 0.00 -> 87.5 mm, vias 0 -> 1
- net +3V3_DIGITAL: track 483.5 -> 560.5 mm, vias 10 -> 17
- net Net-(U8-RUN): track 13.7 -> 65.6 mm, vias 0 -> 4
- net QSPI_CLK: track 0.00 -> 36.6 mm, vias 0 -> 2
- net XOUT: track 38.9 -> 75.0 mm, vias 3 -> 4
- net +3V3_ANALOG: track 98.7 -> 115.7 mm, vias 2 -> 3
- net CURRENT_ALERT: track 0.00 -> 6.85 mm, vias 0 -> 1
- net TFT_MISO: track 68.9 -> 62.1 mm
- net GND: track 717.6 -> 723.1 mm, vias 14 -> 15
- net SWCLK: track 59.1 -> 60.4 mm
- net TFT_SCLK: track 101.7 -> 102.7 mm

Commit message: see..
Routing:
- net I2C_SCL: track 0.00 -> 53.6 mm, vias 0 -> 9
- net QSPI_IO0: track 0.00 -> 53.2 mm, vias 0 -> 4
- net GND: track 723.1 -> 770.2 mm, vias 15 -> 21
- net +3V3_DIGITAL: track 560.5 -> 607.1 mm, vias 17 -> 22
- net BUZZER_CTRL: track 87.5 -> 119.3 mm, vias 1 -> 6
- net CURRENT_ALERT: track 6.85 -> 31.9 mm, vias 1 -> 6
- net Net-(U8-RUN): track 65.6 -> 84.8 mm
- net POT_SPI_SCK: track 149.1 -> 159.4 mm, vias 2 -> 3
- net TFT_MISO: track 62.1 -> 68.9 mm
- net USB_D_M: track 82.7 -> 78.0 mm
- net +1.1V: track 105.1 -> 102.4 mm, vias 5 -> 6
- net ADC_SCLK: track 146.2 -> 147.0 mm

Commit message: removed unnecessary files
Parts:
- added REF**: MountingHole_3mm_Pad_TopBottom, MountingHole:MountingHole_3mm_Pad_TopBottom, F.Cu at (256.3, 155.9)
- added REF**: MountingHole_3mm_Pad_TopBottom, MountingHole:MountingHole_3mm_Pad_TopBottom, F.Cu at (257.0, 25.4)
- added REF**: MountingHole_3mm_Pad_TopBottom, MountingHole:MountingHole_3mm_Pad_TopBottom, F.Cu at (21.2, 26.2)
- added REF**: MountingHole_3mm_Pad_TopBottom, MountingHole:MountingHole_3mm_Pad_TopBottom, F.Cu at (21.2, 155.7)
Routing:
- net ADC_CS: track 101.5 -> 170.9 mm, vias 1 -> 7
- net USB_D_M: track 78.0 -> 84.0 mm, vias 2 -> 5
- net ADC_MISO: track 158.3 -> 160.6 mm
