File: Auralab_Workstation/maincontest.kicad_sch (KiCad schematic)
At the start: 76 parts, among them J1 Conn_Coaxial, J2 TEST_SOCKET, J3 USB_C_Receptacle_USB2.0_16P, J4 Screw_Terminal_01x03, J5 Conn_01x02_Socket, J6 Conn_01x03, J7 Conn_01x14_Socket, Q1 BS170, Q2 BC847, SW1 SW_SPDT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

Commit message: removed unnecessary files
Other:
- note added: "ANALOG FRONTEND"
- note added: "POWER MANAGEMENT"
- note added: "RP2040 Core"
- moved on the sheet: BZ1, C10, C11, C2, C3, C4, C5, C6, C7, C8, C9, Clean_Analog_Filter1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
