File: Auralab_Workstation/Auralab_Workstation.kicad_sch (KiCad schematic)
At the start: 0 parts

Commit message: Updated
Other:
- removed sheet Analog_Front_End
- added sheet Analog_part (pcbwaycontest.kicad_sch)
Changed lines of the file:
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@@
 	(paper "A4")
+	(sheet
+		(at 115.57 26.67)
+		(size 31.75 24.13)
+		(exclude_from_sim no)
+		(in_bom yes)
+		(on_board yes)
+		(dnp no)
+		(fields_autoplaced yes)
+		(stroke
+			(width 0.1524)
+			(type solid)
+		)
+		(fill
+			(color 0 0 0 0.0000)
+		)
+		(property "Sheetname" "Analog_part"
+			(at 115.57 25.9584 0)
+			(effects
+				(font
+					(size 1.27 1.27)
+				)
+				(justify left bottom)
+			)
+		)
+		(property "Sheetfile" "pcbwaycontest.kicad_sch"
+			(at 115.57 51.3846 0)
+			(effects
+				(font
+					(size 1.27 1.27)
+				)
+				(justify left top)
+			)
+		)
+		(instances
+			(project "Auralab_Workstation"
+				(path "/db223ba7-bea5-428e-a07f-3236299d6518"
+					(page "4")
+				)
+			)
+		)
+	)
 	(sheet
 		(at 29.21 26.67)
@@
 				)
 			)
-		)
-	)
-	(sheet
-		(at 116.84 26.67)
-		(size 39.37 22.86)
-		(exclude_from_sim no)
-		(in_bom yes)
-		(on_board yes)
-		(dnp no)
-		(fields_autoplaced yes)
-		(stroke
-			(width 0.1524)
-			(type solid)
-		)
-		(fill
-			(color 0 0 0 0.0000)
-		)
-		(property "Sheetname" "Analog_Front_End"
-			(at 116.84 25.9584 0)
-			(effects
-				(font
-					(size 1.27 1.27)
-				)
-				(justify left bottom)
-			)
-		)
-		(property "Sheetfile" "analog_front_end.kicad_sch"
-			(at 116.84 50.1146 0)
-			(effects
-				(font
-					(size 1.27 1.27)
-				)
-				(justify left top)
-			)
-		)
-		(instances
-			(project "Auralab_Workstation"
-				(path "/db223ba7-bea5-428e-a07f-3236299d6518"
-					(page "4")
-				)
-			)

Commit message: Check ERC
Other:
- removed sheet Analog_part
- added sheet Analog_Frontend (analog_frontend.kicad_sch)
Changed lines of the file:
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@@
 	(paper "A4")
-	(sheet
-		(at 115.57 26.67)
-		(size 31.75 24.13)
-		(exclude_from_sim no)
-		(in_bom yes)
-		(on_board yes)
-		(dnp no)
-		(fields_autoplaced yes)
-		(stroke
-			(width 0.1524)
-			(type solid)
-		)
-		(fill
-			(color 0 0 0 0.0000)
-		)
-		(property "Sheetname" "Analog_part"
-			(at 115.57 25.9584 0)
-			(effects
-				(font
-					(size 1.27 1.27)
-				)
-				(justify left bottom)
-			)
-		)
-		(property "Sheetfile" "pcbwaycontest.kicad_sch"
-			(at 115.57 51.3846 0)
-			(effects
-				(font
-					(size 1.27 1.27)
-				)
-				(justify left top)
-			)
-		)
-		(instances
-			(project "Auralab_Workstation"
-				(path "/db223ba7-bea5-428e-a07f-3236299d6518"
-					(page "4")
-				)
-			)
-		)
-	)
 	(sheet
 		(at 29.21 26.67)
@@
 				)
 			)
+		)
+	)
+	(sheet
+		(at 114.3 26.67)
+		(size 41.91 22.86)
+		(exclude_from_sim no)
+		(in_bom yes)
+		(on_board yes)
+		(dnp no)
+		(fields_autoplaced yes)
+		(stroke
+			(width 0.1524)
+			(type solid)
+		)
+		(fill
+			(color 0 0 0 0.0000)
+		)
+		(property "Sheetname" "Analog_Frontend"
+			(at 114.3 25.9584 0)
+			(effects
+				(font
+					(size 1.27 1.27)
+				)
+				(justify left bottom)
+			)
+		)
+		(property "Sheetfile" "analog_frontend.kicad_sch"
+			(at 114.3 50.1146 0)
+			(effects
+				(font
+					(size 1.27 1.27)
+				)
+				(justify left top)
+			)
+		)
+		(instances
+			(project "Auralab_Workstation"
+				(path "/db223ba7-bea5-428e-a07f-3236299d6518"
+					(page "4")
+				)
+			)

Commit message: uPDATED AURALAB workstation
Parts:
- added BZ2: Buzzer, Buzzer_Beeper:Buzzer_CUI_CPT-9019S-SMT, symbol Device:Buzzer
- added C13: 10uF, Capacitor_Tantalum_SMD:CP_EIA-6032-28_Kemet-C_HandSolder, symbol Device:C_Polarized
- added C14: 47nF, Capacitor_SMD:C_0805_2012Metric_Pad1.18x1.45mm_HandSolder, symbol Device:C
- added C15, C16, C17: 10uF, Capacitor_SMD:C_0805_2012Metric_Pad1.18x1.45mm_HandSolder, symbol Device:C
- added C18, C19: 0.1uF, Capacitor_SMD:C_0805_2012Metric, symbol Device:C
- added C20: 1uF, Capacitor_SMD:C_0805_2012Metric_Pad1.18x1.45mm_HandSolder, symbol Device:C
- added C21, C22: 27pF, Capacitor_SMD:C_0805_2012Metric_Pad1.18x1.45mm_HandSolder, symbol Device:C
- added C23, C24, Clean_Analog_Filter2, Digital_Filter2, Regulator_Filter2: 100nF, Capacitor_SMD:C_0805_2012Metric_Pad1.18x1.45mm_HandSolder, symbol Device:C
- added D10, D11, D12: MBR0520, Diode_SMD:D_SOD-123, symbol Diode:MBR0520
- added D13: RED_LED, LED_SMD:LED_0805_2012Metric_Pad1.15x1.40mm_HandSolder, symbol Device:LED
- added D14: GREEN_LED, LED_SMD:LED_0805_2012Metric_Pad1.15x1.40mm_HandSolder, symbol Device:LED
- added D15, D16: 1N4148W, Diode_SMD:D_SOD-123, symbol Diode:1N4148W
- added D17: POWER_ON_LED, LED_SMD:LED_0805_2012Metric_Pad1.15x1.40mm_HandSolder, symbol Device:LED
- added D18: LED, LED_SMD:LED_0805_2012Metric_Pad1.15x1.40mm_HandSolder, symbol Device:LED
- added F2: Polyfuse, Fuse:Fuse_1206_3216Metric, symbol Device:Polyfuse
- added FB2: FerriteBead, Inductor_SMD:L_0805_2012Metric_Pad1.15x1.40mm_HandSolder, symbol Device:FerriteBead
- added J10: Conn_01x02_Socket, Connector_JST:JST_PH_B2B-PH-K_1x02_P2.00mm_Vertical, symbol Connector:Conn_01x02_Socket
- added J11: Conn_Coaxial, Connector_Coaxial:BNC_Amphenol_B6252HB-NPP3G-50_Horizontal, symbol Connector:Conn_Coaxial
- added J12: TEST_SOCKET, TerminalBlock_Phoenix:TerminalBlock_Phoenix_MPT-0,5-3-2.54_1x03_P2.54mm_Horizontal, symbol Connector:Screw_Terminal_01x03
- added J13: Conn_01x03, Connector_PinHeader_2.54mm:PinHeader_1x03_P2.54mm_Vertical, symbol Connector_Generic:Conn_01x03
- added J14: Conn_01x14_Socket, Connector_PinSocket_2.54mm:PinSocket_1x14_P2.54mm_Vertical, symbol Connector:Conn_01x14_Socket
- added J8: USB_C_Receptacle_USB2.0_16P, Connector_USB:USB_C_Receptacle_HRO_TYPE-C-31-M-12, symbol Connector:USB_C_Receptacle_USB2.0_16P
- added J9: Screw_Terminal_01x03, TerminalBlock:TerminalBlock_MaiXu_MX126-5.0-03P_1x03_P5.00mm, symbol Connector:Screw_Terminal_01x03
- added L3, L4: 4.7uH, Inductor_SMD:L_6.3x6.3_H3, symbol Device:L
- added Q3: BS170, Package_TO_SOT_THT:TO-92_Inline, symbol Transistor_FET:BS170
- added Q4: BC847, Package_TO_SOT_SMD:SOT-23, symbol Transistor_BJT:BC847
- added R24, R25: 5.1k Ohm, Resistor_SMD:R_0805_2012Metric_Pad1.20x1.40mm_HandSolder, symbol Device:R
- added R26, R27: 1M Ohm, Resistor_SMD:R_0805_2012Metric_Pad1.20x1.40mm_HandSolder, symbol Device:R
- added R28, R29, R38, R39: 220 Ohm, Resistor_SMD:R_0805_2012Metric_Pad1.20x1.40mm_HandSolder, symbol Device:R
- added R30: R_prog = 1.2k, Resistor_SMD:R_0805_2012Metric_Pad1.20x1.40mm_HandSolder, symbol Device:R
- added R31: 1M Ohm, Resistor_SMD:R_0805_2012Metric, symbol Device:R
- added R32, R35: 10k Ohm, Resistor_SMD:R_0805_2012Metric, symbol Device:R
- added R33: 1k Ohm, Resistor_SMD:R_0805_2012Metric, symbol Device:R
- added R34: 3.3k Ohm, Resistor_SMD:R_0805_2012Metric, symbol Device:R
- added R36: 10 Ohm, Resistor_SMD:R_0805_2012Metric, symbol Device:R
- added R37: 0.1 Ohm, Resistor_SMD:R_0805_2012Metric, symbol Device:R
- added R40: 1k Ohm, Resistor_SMD:R_0805_2012Metric_Pad1.20x1.40mm_HandSolder, symbol Device:R
- added R41, R42: 27 Ohm, Resistor_SMD:R_0805_2012Metric_Pad1.20x1.40mm_HandSolder, symbol Device:R
- added R43: 10 Ohm, Resistor_SMD:R_0805_2012Metric_Pad1.20x1.40mm_HandSolder, symbol Device:R
- added R44: 10k Ohm, Resistor_SMD:R_0805_2012Metric_Pad1.20x1.40mm_HandSolder, symbol Device:R
- added R45: 100 Ohm, Resistor_SMD:R_0805_2012Metric_Pad1.20x1.40mm_HandSolder, symbol Device:R
- added R46: 1k, Resistor_SMD:R_0805_2012Metric_Pad1.20x1.40mm_HandSolder, symbol Device:R
- added SW4: SW_SPDT, Button_Switch_SMD:SW_SPDT_PCM12, symbol Switch:SW_SPDT
- added SW5: RotaryEncoder_Switch, Rotary_Encoder:RotaryEncoder_Alps_EC11E-Switch_Vertical_H20mm, symbol Device:RotaryEncoder_Switch
- added SW6: SW_Push, Button_Switch_THT:SW_PUSH-12mm_Wuerth-430476085716, symbol Switch:SW_Push
- added U12: TPS65131RGE, Package_DFN_QFN:VQFN-24-1EP_4x4mm_P0.5mm_EP2.45x2.45mm_ThermalVias, symbol Regulator_Switching:TPS65131RGE
- added U13: USBLC6-2SC6, Package_TO_SOT_SMD:SOT-23-6, symbol Power_Protection:USBLC6-2SC6
- added U14: AP2112K-3.3, Package_TO_SOT_SMD:SOT-23-5, symbol Regulator_Linear:AP2112K-3.3
- added U15: TP4056-42-ESOP8, Package_SO:SOIC-8-1EP_3.9x4.9mm_P1.27mm_EP2.41x3.3mm_ThermalVias, symbol Battery_Management:TP4056-42-ESOP8
- added U16: MCP42010, Package_SO:SOIC-14_3.9x8.7mm_P1.27mm, symbol Potentiometer_Digital:MCP42010
- added U17: TL072, Package_SO:SOIC-8_3.9x4.9mm_P1.27mm, symbol Amplifier_Operational:TL072
- added U18: REF3033, Package_TO_SOT_SMD:SOT-23, symbol Reference_Voltage:REF3033
- added U19: MCP3201, Package_SO:SOIC-8_3.9x4.9mm_P1.27mm, symbol Analog_ADC:MCP3201
- added U20: INA226, Package_SO:VSSOP-10_3x3mm_P0.5mm, symbol Sensor_Energy:INA226
- added U21: RP2040, Package_DFN_QFN:QFN-56-1EP_7x7mm_P0.4mm_EP3.2x3.2mm, symbol MCU_RaspberryPi:RP2040
- added U22: W25Q128JVS, Package_SO:SOIC-8_5.3x5.3mm_P1.27mm, symbol Memory_Flash:W25Q128JVS
- added Y2: Crystal_GND24, Crystal:Crystal_SMD_3225-4Pin_3.2x2.5mm_HandSoldering, symbol Device:Crystal_GND24
Connections:
- new net: BZ2.2 (-), Q4.3 (C)
- new net: J14.8 (Pin_8), R45.2
- new net: Q4.1 (B), R40.2
- new net: R44.2, SW6.1, U21.26 (RUN)
- new net: D14.2 (A), R29.2
- new net: D10.2 (A), L3.1, U12.7 (BSW)
- new net: J8.A5 (CC1), R24.1
- new net: J8.B5 (CC2), R25.1
- new net: R33.1, U17.1, U17.2 (-)
- new net: D12.1 (K), L4.2, U12.13 (OUTN), U12.14 (OUTN), U12.18 (CN)
- new net: F2.2, FB2.1
- new net: D11.1 (K), F2.1
- new net: C18.2, R31.1, SW4.3 (C)
- new net: D17.1 (K), R38.2
- new net: Q3.1 (D), R37.2
- new net: J11.1 (In), SW4.2 (B)
- new net: D13.1 (K), U15.7 (~{CHRG})
- new net: D13.2 (A), R28.2
- new net: R34.1, R35.1, U17.6 (-)
- new net: D18.1 (K), R39.2
- new net: D14.1 (K), U15.6 (~{STDBY})
- new net: C18.1, SW4.1 (A)
- new net: R30.1, U15.2 (PROG)
- new net +1.1V: C20.1, U21.23 (DVDD), U21.45 (VREG_VOUT), U21.50 (DVDD)
- new net +3V3_ANALOG: Clean_Analog_Filter2.1, R43.2, U21.43 (ADC_AVDD)
- new net +3V3_DIGITAL: BZ2.1 (+), C16.1, C19.1, C23.1, D15.1 (K), D17.2 (A), Digital_Filter2.1, J14.1 (Pin_1), R43.1, R44.1, Regulator_Filter2.1, U12.10 (ENN), U12.8 (ENP), U14.5 (VOUT), U16.11 (~{RS}), U16.12 (~{SHDN}), U16.14 (VDD), U18.1 (IN), U19.8 (Vdd), U20.6 (VS), U21.1 (IOVDD), U21.10 (IOVDD), U21.22 (IOVDD), U21.33 (IOVDD), U21.42 (IOVDD), U21.44 (VREG_IN), U21.48 (USB_VDD), U21.49 (IOVDD), U22.8 (VCC)
- new net +5V_RAW: FB2.2, R28.1, R29.1, R45.1, U15.4 (V_{CC}), U15.8 (CE)
- new net +IN_ADC: D15.2 (A), D16.1 (K), R33.2, U19.2 (IN+)
- new net +Vout: C13.1, D10.1 (K), J9.1 (Pin_1), R26.1, U12.23 (VPOS), U17.8 (V+)
- new net -Vout: D12.2 (A), J9.3 (Pin_3), R27.2, U12.15 (VNEG), U17.4 (V-)
- new net A4: D11.2 (A), J8.A4 (VBUS), J8.A9 (VBUS), J8.B4 (VBUS), J8.B9 (VBUS)
- new net A6: J8.A6 (D+), U13.3 (I/O2)
- new net A7: J8.A7 (D-), U13.1 (I/O1)
- new net ADC_CS: U19.5 (~{CS}/SHDN), U21.8 (GPIO6)
- new net ADC_MISO: U19.6 (Dout), U21.5 (GPIO3)
- new net ADC_SCLK: U19.7 (CLK), U21.4 (GPIO2)
- new net ALERT_LED: D18.2 (A), U21.35 (GPIO23)
- new net BUZZER_CTRL: R40.1, U21.11 (GPIO8)
- new net CURRENT_ALERT: U20.3 (~{Alert}), U21.12 (GPIO9)
- new net CURRENT_IN: J12.2 (Pin_2), R36.1, R37.1, U20.10 (Vin+), U20.8 (Vbus)
- new net FBN: R27.1, U12.16 (FBN), U16.5 (PB1), U16.6 (PW1)
- new net FBP: R26.2, U12.22 (FBP), U16.8 (PA0), U16.9 (PW0)
- new net GND: C15.1, C16.2, C17.2, C19.2, C20.2, C21.2, C22.2, C23.2, C24.2, Clean_Analog_Filter2.2, Digital_Filter2.2, J10.2 (Pin_2), J13.3 (Pin_3), J14.2 (Pin_2), J8.A1 (GND), J8.A12 (GND), J8.B1 (GND), J8.B12 (GND), J8.S1 (SHIELD), L4.1, Q4.2 (E), R24.2, R25.2, R30.2, R38.1, R39.1, Regulator_Filter2.2, SW5.C, SW5.S2, SW6.2, U12.11 (PSN), U12.2 (PGND), U12.21 (CP), U12.25 (EP), U12.3 (PGND), U12.9 (PSP), U13.2 (GND), U14.2 (GND), U15.1 (TEMP), U15.3 (GND), U15.9 (EPAD), U19.4 (Vss), U20.1 (A1), U20.2 (A0), U20.7 (GND), U21.57 (GND), U22.4 (GND), Y2.2, Y2.4
- new net GNDA: C13.2, C14.2, D16.2 (A), J11.2 (Ext), J12.3 (Pin_3), J9.2 (Pin_2), Q3.3 (S), R32.2, R34.2, R36.2, U12.19 (AGND), U16.10 (PB0), U16.4 (VSS), U18.3 (GND), U19.3 (IN-), U20.9 (Vin-)
- new net I2C_SCL: U20.5 (SCL), U21.7 (GPIO5)
- new net I2C_SDA: U20.4 (SDA), U21.6 (GPIO4)
- new net Non-inv Input OpAmp: R31.2, R32.1, U17.3 (+)
- new net POT_SPI_CS: U16.1 (~{CS}), U21.15 (GPIO12)
- new net POT_SPI_MOSI: U16.3 (SI), U21.17 (GPIO14)
- new net POT_SPI_SCK: U16.2 (SCK), U21.16 (GPIO13)
- new net QSPI_CLK: U21.52 (QSPI_SCLK), U22.6 (CLK)
- new net QSPI_CS: U21.56 (QSPI_SS), U22.1 (~{CS})
- new net QSPI_IO0: U21.53 (QSPI_SD0), U22.5 (DI/IO_{0})
- new net QSPI_IO1: U21.55 (QSPI_SD1), U22.2 (DO/IO_{1})
- new net QSPI_IO2: U21.54 (QSPI_SD2), U22.3 (~{WP}/IO_{2})
- new net QSPI_IO3: U21.51 (QSPI_SD3), U22.7 (~{HOLD}/~{RESET}/IO_{3})
- new net RANGE_SELECT: Q3.2 (G), U21.9 (GPIO7)
- new net ROT_A: SW5.A, U21.32 (GPIO21)
- new net ROT_B: SW5.B, U21.14 (GPIO11)
- new net ROT_SW: SW5.S1, U21.34 (GPIO22)
- new net SWCLK: J13.1 (Pin_1), U21.24 (SWCLK)
- new net SWD: J13.2 (Pin_2), U21.25 (SWD)
- new net SWEEP_PWM: R46.1, U21.13 (GPIO10)
- new net TFT_CS: J14.3 (Pin_3), U21.29 (GPIO18)
- new net TFT_DC: J14.5 (Pin_5), U21.30 (GPIO19)
- new net TFT_MISO: J14.9 (Pin_9), U21.18 (GPIO15)
- new net TFT_MOSI: J14.6 (Pin_6), U21.28 (GPIO17)
- new net TFT_RST: J14.4 (Pin_4), U21.31 (GPIO20)
- new net TFT_SCLK: J14.7 (Pin_7), U21.27 (GPIO16)
- new net USB_DM: R42.1, U13.6 (I/O1)
- new net USB_DP: R41.1, U13.4 (I/O2)
- new net USB_D_M: R42.2, U21.46 (USB_DM)
- new net USB_D_P: R41.2, U21.47 (USB_DP)
- new net VBUS_SYSTEM: C15.2, C17.1, J10.1 (Pin_1), L3.2, U12.1 (INP), U12.24 (INP), U12.4 (VIN), U12.5 (INN), U12.6 (INN), U14.1 (VIN), U14.3 (EN), U15.5 (BAT)
- new net V_SWEEP: J12.1 (Pin_1), R35.2, U17.7
- new net V_filtered: C24.1, R46.2, U17.5 (+)
- new net Vref: C14.1, U12.17 (VREF), U16.7 (PA1)
- new net Vref_ADC: U18.2 (OUT), U19.1 (Vref)
- new net XIN: C21.1, U21.20 (XIN), Y2.1
- new net XOUT: C22.1, U21.21 (XOUT), Y2.3
- no-connect marks 0 -> 20

Commit message: pcb..
Parts:
- renumbered J11 to J1
Changed lines of the file:
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@@
 		(dnp no)
 		(fields_autoplaced yes)
-		(property "Reference" "J11"
-			(at 30.48 186.9831 0)
+		(property "Reference" "J1"
+			(at 34.6074 181.61 0)
 			(effects
 				(font
 					(size 1.27 1.27)
 				)
-				(justify left)
 			)
 		)
 		(property "Value" "Conn_Coaxial"
-			(at 30.48 189.5231 0)
+			(at 34.6074 184.15 0)
 			(effects
 				(font
 					(size 1.27 1.27)
 				)
-				(justify left)
 			)
 		)
@@
 			(project "Auralab_Workstation"
 				(path "/db223ba7-bea5-428e-a07f-3236299d6518"
-					(reference "J11")
+					(reference "J1")
 					(unit 1)
 				)

Commit message: Made few changes check
Parts:
- removed BZ2: Buzzer, Buzzer_Beeper:Buzzer_CUI_CPT-9019S-SMT, symbol Device:Buzzer
- removed C13: 10uF, Capacitor_Tantalum_SMD:CP_EIA-6032-28_Kemet-C_HandSolder, symbol Device:C_Polarized
- removed C14: 47nF, Capacitor_SMD:C_0805_2012Metric_Pad1.18x1.45mm_HandSolder, symbol Device:C
- removed C15, C16, C17: 10uF, Capacitor_SMD:C_0805_2012Metric_Pad1.18x1.45mm_HandSolder, symbol Device:C
- removed C18, C19: 0.1uF, Capacitor_SMD:C_0805_2012Metric, symbol Device:C
- removed C20: 1uF, Capacitor_SMD:C_0805_2012Metric_Pad1.18x1.45mm_HandSolder, symbol Device:C
- removed C21, C22: 27pF, Capacitor_SMD:C_0805_2012Metric_Pad1.18x1.45mm_HandSolder, symbol Device:C
- removed C23, C24, Clean_Analog_Filter2, Digital_Filter2, Regulator_Filter2: 100nF, Capacitor_SMD:C_0805_2012Metric_Pad1.18x1.45mm_HandSolder, symbol Device:C
- removed D10, D11, D12: MBR0520, Diode_SMD:D_SOD-123, symbol Diode:MBR0520
- removed D13: RED_LED, LED_SMD:LED_0805_2012Metric_Pad1.15x1.40mm_HandSolder, symbol Device:LED
- removed D14: GREEN_LED, LED_SMD:LED_0805_2012Metric_Pad1.15x1.40mm_HandSolder, symbol Device:LED
- removed D15, D16: 1N4148W, Diode_SMD:D_SOD-123, symbol Diode:1N4148W
- removed D17: POWER_ON_LED, LED_SMD:LED_0805_2012Metric_Pad1.15x1.40mm_HandSolder, symbol Device:LED
- removed D18: LED, LED_SMD:LED_0805_2012Metric_Pad1.15x1.40mm_HandSolder, symbol Device:LED
- removed F2: Polyfuse, Fuse:Fuse_1206_3216Metric, symbol Device:Polyfuse
- removed FB2: FerriteBead, Inductor_SMD:L_0805_2012Metric_Pad1.15x1.40mm_HandSolder, symbol Device:FerriteBead
- removed J10: Conn_01x02_Socket, Connector_JST:JST_PH_B2B-PH-K_1x02_P2.00mm_Vertical, symbol Connector:Conn_01x02_Socket
- removed J12: TEST_SOCKET, TerminalBlock_Phoenix:TerminalBlock_Phoenix_MPT-0,5-3-2.54_1x03_P2.54mm_Horizontal, symbol Connector:Screw_Terminal_01x03
- removed J13: Conn_01x03, Connector_PinHeader_2.54mm:PinHeader_1x03_P2.54mm_Vertical, symbol Connector_Generic:Conn_01x03
- removed J14: Conn_01x14_Socket, Connector_PinSocket_2.54mm:PinSocket_1x14_P2.54mm_Vertical, symbol Connector:Conn_01x14_Socket
- removed J8: USB_C_Receptacle_USB2.0_16P, Connector_USB:USB_C_Receptacle_HRO_TYPE-C-31-M-12, symbol Connector:USB_C_Receptacle_USB2.0_16P
- removed J9: Screw_Terminal_01x03, TerminalBlock:TerminalBlock_MaiXu_MX126-5.0-03P_1x03_P5.00mm, symbol Connector:Screw_Terminal_01x03
- removed L3, L4: 4.7uH, Inductor_SMD:L_6.3x6.3_H3, symbol Device:L
- removed Q3: BS170, Package_TO_SOT_THT:TO-92_Inline, symbol Transistor_FET:BS170
- removed Q4: BC847, Package_TO_SOT_SMD:SOT-23, symbol Transistor_BJT:BC847
- removed R24, R25: 5.1k Ohm, Resistor_SMD:R_0805_2012Metric_Pad1.20x1.40mm_HandSolder, symbol Device:R
- removed R26, R27: 1M Ohm, Resistor_SMD:R_0805_2012Metric_Pad1.20x1.40mm_HandSolder, symbol Device:R
- removed R28, R29, R38, R39: 220 Ohm, Resistor_SMD:R_0805_2012Metric_Pad1.20x1.40mm_HandSolder, symbol Device:R
- removed R30: R_prog = 1.2k, Resistor_SMD:R_0805_2012Metric_Pad1.20x1.40mm_HandSolder, symbol Device:R
- removed R31: 1M Ohm, Resistor_SMD:R_0805_2012Metric, symbol Device:R
- removed R32, R35: 10k Ohm, Resistor_SMD:R_0805_2012Metric, symbol Device:R
- removed R33: 1k Ohm, Resistor_SMD:R_0805_2012Metric, symbol Device:R
- removed R34: 3.3k Ohm, Resistor_SMD:R_0805_2012Metric, symbol Device:R
- removed R36: 10 Ohm, Resistor_SMD:R_0805_2012Metric, symbol Device:R
- removed R37: 0.1 Ohm, Resistor_SMD:R_0805_2012Metric, symbol Device:R
- removed R40: 1k Ohm, Resistor_SMD:R_0805_2012Metric_Pad1.20x1.40mm_HandSolder, symbol Device:R
- removed R41, R42: 27 Ohm, Resistor_SMD:R_0805_2012Metric_Pad1.20x1.40mm_HandSolder, symbol Device:R
- removed R43: 10 Ohm, Resistor_SMD:R_0805_2012Metric_Pad1.20x1.40mm_HandSolder, symbol Device:R
- removed R44: 10k Ohm, Resistor_SMD:R_0805_2012Metric_Pad1.20x1.40mm_HandSolder, symbol Device:R
- removed R45: 100 Ohm, Resistor_SMD:R_0805_2012Metric_Pad1.20x1.40mm_HandSolder, symbol Device:R
- removed R46: 1k, Resistor_SMD:R_0805_2012Metric_Pad1.20x1.40mm_HandSolder, symbol Device:R
- removed SW4: SW_SPDT, Button_Switch_SMD:SW_SPDT_PCM12, symbol Switch:SW_SPDT
- removed SW5: RotaryEncoder_Switch, Rotary_Encoder:RotaryEncoder_Alps_EC11E-Switch_Vertical_H20mm, symbol Device:RotaryEncoder_Switch
- removed SW6: SW_Push, Button_Switch_THT:SW_PUSH-12mm_Wuerth-430476085716, symbol Switch:SW_Push
- removed U12: TPS65131RGE, Package_DFN_QFN:VQFN-24-1EP_4x4mm_P0.5mm_EP2.45x2.45mm_ThermalVias, symbol Regulator_Switching:TPS65131RGE
- removed U13: USBLC6-2SC6, Package_TO_SOT_SMD:SOT-23-6, symbol Power_Protection:USBLC6-2SC6
- removed U14: AP2112K-3.3, Package_TO_SOT_SMD:SOT-23-5, symbol Regulator_Linear:AP2112K-3.3
- removed U15: TP4056-42-ESOP8, Package_SO:SOIC-8-1EP_3.9x4.9mm_P1.27mm_EP2.41x3.3mm_ThermalVias, symbol Battery_Management:TP4056-42-ESOP8
- removed U16: MCP42010, Package_SO:SOIC-14_3.9x8.7mm_P1.27mm, symbol Potentiometer_Digital:MCP42010
- removed U17: TL072, Package_SO:SOIC-8_3.9x4.9mm_P1.27mm, symbol Amplifier_Operational:TL072
- removed U18: REF3033, Package_TO_SOT_SMD:SOT-23, symbol Reference_Voltage:REF3033
- removed U19: MCP3201, Package_SO:SOIC-8_3.9x4.9mm_P1.27mm, symbol Analog_ADC:MCP3201
- removed U20: INA226, Package_SO:VSSOP-10_3x3mm_P0.5mm, symbol Sensor_Energy:INA226
- removed U21: RP2040, Package_DFN_QFN:QFN-56-1EP_7x7mm_P0.4mm_EP3.2x3.2mm, symbol MCU_RaspberryPi:RP2040
- removed U22: W25Q128JVS, Package_SO:SOIC-8_5.3x5.3mm_P1.27mm, symbol Memory_Flash:W25Q128JVS
- removed Y2: Crystal_GND24, Crystal:Crystal_SMD_3225-4Pin_3.2x2.5mm_HandSoldering, symbol Device:Crystal_GND24
- added BZ1: Buzzer, Buzzer_Beeper:Buzzer_CUI_CPT-9019S-SMT, symbol Device:Buzzer
- added C1, C12: 0.1uF, Capacitor_SMD:C_0805_2012Metric, symbol Device:C
- added C10, C9, Clean_Analog_Filter1, Digital_Filter1, Regulator_Filter1: 100nF, Capacitor_SMD:C_0805_2012Metric_Pad1.18x1.45mm_HandSolder, symbol Device:C
- added C11, C3, C5: 10uF, Capacitor_SMD:C_0805_2012Metric_Pad1.18x1.45mm_HandSolder, symbol Device:C
- added C2: 10uF, Capacitor_Tantalum_SMD:CP_EIA-6032-28_Kemet-C_HandSolder, symbol Device:C_Polarized
- added C4: 47nF, Capacitor_SMD:C_0805_2012Metric_Pad1.18x1.45mm_HandSolder, symbol Device:C
- added C6: 1uF, Capacitor_SMD:C_0805_2012Metric_Pad1.18x1.45mm_HandSolder, symbol Device:C
- added C7, C8: 27pF, Capacitor_SMD:C_0805_2012Metric_Pad1.18x1.45mm_HandSolder, symbol Device:C
- added D1, D9: 1N4148W, Diode_SMD:D_SOD-123, symbol Diode:1N4148W
- added D2, D3, D6: MBR0520, Diode_SMD:D_SOD-123, symbol Diode:MBR0520
- added D4: POWER_ON_LED, LED_SMD:LED_0805_2012Metric_Pad1.15x1.40mm_HandSolder, symbol Device:LED
- added D5: LED, LED_SMD:LED_0805_2012Metric_Pad1.15x1.40mm_HandSolder, symbol Device:LED
- added D7: RED_LED, LED_SMD:LED_0805_2012Metric_Pad1.15x1.40mm_HandSolder, symbol Device:LED
- added D8: GREEN_LED, LED_SMD:LED_0805_2012Metric_Pad1.15x1.40mm_HandSolder, symbol Device:LED
- added F1: Polyfuse, Fuse:Fuse_1206_3216Metric, symbol Device:Polyfuse
- added FB1: FerriteBead, Inductor_SMD:L_0805_2012Metric, symbol Device:FerriteBead
- added J2: TEST_SOCKET, TerminalBlock_Phoenix:TerminalBlock_Phoenix_MPT-0,5-3-2.54_1x03_P2.54mm_Horizontal, symbol Connector:Screw_Terminal_01x03
- added J3: USB_C_Receptacle_USB2.0_16P, Connector_USB:USB_C_Receptacle_HRO_TYPE-C-31-M-12, symbol Connector:USB_C_Receptacle_USB2.0_16P
- added J4: Screw_Terminal_01x03, TerminalBlock:TerminalBlock_MaiXu_MX126-5.0-03P_1x03_P5.00mm, symbol Connector:Screw_Terminal_01x03
- added J5: Conn_01x02_Socket, Connector_JST:JST_PH_B2B-PH-K_1x02_P2.00mm_Vertical, symbol Connector:Conn_01x02_Socket
- added J6: Conn_01x03, Connector_PinHeader_2.54mm:PinHeader_1x03_P2.54mm_Vertical, symbol Connector_Generic:Conn_01x03
- added J7: Conn_01x14_Socket, Connector_PinSocket_2.54mm:PinSocket_1x14_P2.54mm_Vertical, symbol Connector:Conn_01x14_Socket
- added L1, L2: 4.7uH, Inductor_SMD:L_6.3x6.3_H3, symbol Device:L
- added Q1: BS170, Package_TO_SOT_THT:TO-92_Inline, symbol Transistor_FET:BS170
- added Q2: BC847, Package_TO_SOT_SMD:SOT-23, symbol Transistor_BJT:BC847
- added R1: 1M Ohm, Resistor_SMD:R_0805_2012Metric, symbol Device:R
- added R10, R11, R12, R9: 220 Ohm, Resistor_SMD:R_0805_2012Metric_Pad1.20x1.40mm_HandSolder, symbol Device:R
- added R13: 1k Ohm, Resistor_SMD:R_0805_2012Metric_Pad1.20x1.40mm_HandSolder, symbol Device:R
- added R14, R15: 27 Ohm, Resistor_SMD:R_0805_2012Metric_Pad1.20x1.40mm_HandSolder, symbol Device:R
- added R16: 10 Ohm, Resistor_SMD:R_0805_2012Metric_Pad1.20x1.40mm_HandSolder, symbol Device:R
- added R17: 10k Ohm, Resistor_SMD:R_0805_2012Metric_Pad1.20x1.40mm_HandSolder, symbol Device:R
- added R18: R_prog = 1.2k, Resistor_SMD:R_0805_2012Metric_Pad1.20x1.40mm_HandSolder, symbol Device:R
- added R19: 100 Ohm, Resistor_SMD:R_0805_2012Metric_Pad1.20x1.40mm_HandSolder, symbol Device:R
- added R2: 0.1 Ohm, Resistor_SMD:R_0805_2012Metric, symbol Device:R
- added R20: 1k Ohm, Resistor_SMD:R_0805_2012Metric, symbol Device:R
- added R21: 3.3k Ohm, Resistor_SMD:R_0805_2012Metric, symbol Device:R
- added R22: 1k, Resistor_SMD:R_0805_2012Metric_Pad1.20x1.40mm_HandSolder, symbol Device:R
- added R23, R3: 10k Ohm, Resistor_SMD:R_0805_2012Metric, symbol Device:R
- added R4: 10 Ohm, Resistor_SMD:R_0805_2012Metric, symbol Device:R
- added R5, R6: 5.1k Ohm, Resistor_SMD:R_0805_2012Metric_Pad1.20x1.40mm_HandSolder, symbol Device:R
- added R7, R8: 1M Ohm, Resistor_SMD:R_0805_2012Metric_Pad1.20x1.40mm_HandSolder, symbol Device:R
- added SW1: SW_SPDT, Button_Switch_SMD:SW_SPDT_PCM12, symbol Switch:SW_SPDT
- added SW2: RotaryEncoder_Switch, Rotary_Encoder:RotaryEncoder_Alps_EC11E-Switch_Vertical_H20mm, symbol Device:RotaryEncoder_Switch
- added SW3: SW_Push, Button_Switch_THT:SW_PUSH-12mm_Wuerth-430476085716, symbol Switch:SW_Push
- added U1: TL072, Package_SO:SOIC-8_3.9x4.9mm_P1.27mm, symbol Amplifier_Operational:TL072
- added U10: TP4056-42-ESOP8, Package_SO:SOIC-8-1EP_3.9x4.9mm_P1.27mm_EP2.41x3.3mm_ThermalVias, symbol Battery_Management:TP4056-42-ESOP8
- added U11: MCP42010, Package_SO:SOIC-14_3.9x8.7mm_P1.27mm, symbol Potentiometer_Digital:MCP42010
- added U2: MCP3201, Package_SO:SOIC-8_3.9x4.9mm_P1.27mm, symbol Analog_ADC:MCP3201
- added U3: REF3033, Package_TO_SOT_SMD:SOT-23, symbol Reference_Voltage:REF3033
- added U4: TPS65131RGE, Package_DFN_QFN:VQFN-24-1EP_4x4mm_P0.5mm_EP2.45x2.45mm_ThermalVias, symbol Regulator_Switching:TPS65131RGE
- added U5: INA226, Package_SO:MSOP-10_3x3mm_P0.5mm, symbol Sensor_Energy:INA226
- added U6: USBLC6-2SC6, Package_TO_SOT_SMD:SOT-23-6, symbol Power_Protection:USBLC6-2SC6
- added U7: AP2112K-3.3, Package_TO_SOT_SMD:SOT-23-5, symbol Regulator_Linear:AP2112K-3.3
- added U8: RP2040, Package_DFN_QFN:QFN-56-1EP_7x7mm_P0.4mm_EP3.2x3.2mm, symbol MCU_RaspberryPi:RP2040
- added U9: W25Q128JVS, Package_SO:SOIC-8_5.3x5.3mm_P1.27mm, symbol Memory_Flash:W25Q128JVS
- added Y1: Crystal_GND24, Crystal:Crystal_SMD_3225-4Pin_3.2x2.5mm_HandSoldering, symbol Device:Crystal_GND24
Connections:
- net +1.1V: now also C6.1, U8.23 (DVDD), U8.45 (VREG_VOUT), U8.50 (DVDD)
- net +3V3_ANALOG: now also Clean_Analog_Filter1.1, R16.2, U8.43 (ADC_AVDD)
- net +3V3_DIGITAL: now also BZ1.1 (+), C12.1, C5.1, C9.1, D4.2 (A), D9.1 (K), Digital_Filter1.1, J7.1 (Pin_1), R16.1, R17.1, Regulator_Filter1.1, U11.11 (~{RS}), U11.12 (~{SHDN}), U11.14 (VDD), U2.8 (Vdd), U3.1 (IN), U4.10 (ENN), U4.8 (ENP), U5.6 (VS), U7.5 (VOUT), U8.1 (IOVDD), U8.10 (IOVDD), U8.22 (IOVDD), U8.33 (IOVDD), U8.42 (IOVDD), U8.44 (VREG_IN), U8.48 (USB_VDD), U8.49 (IOVDD), U9.8 (VCC)
- net +5V_RAW: now also FB1.2, R10.1, R19.1, R9.1, U10.4 (V_{CC}), U10.8 (CE)
- net +IN_ADC: now also D1.1 (K), D9.2 (A), R20.2, U2.2 (IN+)
- net +Vout: now also C2.1, D2.1 (K), J4.1 (Pin_1), R7.1, U1.8 (V+), U4.23 (VPOS)
- net -Vout: now also D3.2 (A), J4.3 (Pin_3), R8.2, U1.4 (V-), U4.15 (VNEG)
- net A4: now also D6.2 (A), J3.A4 (VBUS), J3.A9 (VBUS), J3.B4 (VBUS), J3.B9 (VBUS)
- net A6: now also J3.A6 (D+), U6.3 (I/O2)
- net A7: now also J3.A7 (D-), U6.1 (I/O1)
- net ADC_CS: now also U2.5 (~{CS}/SHDN), U8.8 (GPIO6)
- net ADC_MISO: now also U2.6 (Dout), U8.5 (GPIO3)
- net ADC_SCLK: now also U2.7 (CLK), U8.4 (GPIO2)
- net ALERT_LED: now also D5.2 (A), U8.35 (GPIO23)
- net BUZZER_CTRL: now also R13.1, U8.11 (GPIO8)
- net CURRENT_ALERT: now also U5.3 (~{Alert}), U8.12 (GPIO9)
- net CURRENT_IN: now also J2.2 (Pin_2), R2.1, R4.1, U5.10 (Vin+), U5.8 (Vbus)
- net FBN: now also R8.1, U11.5 (PB1), U11.6 (PW1), U4.16 (FBN)
- net FBP: now also R7.2, U11.8 (PA0), U11.9 (PW0), U4.22 (FBP)
- net GND: now also C10.2, C11.2, C12.2, C3.1, C5.2, C6.2, C7.2, C8.2, C9.2, Clean_Analog_Filter1.2, Digital_Filter1.2, J3.A1 (GND), J3.A12 (GND), J3.B1 (GND), J3.B12 (GND), J3.S1 (SHIELD), J5.2 (Pin_2), J6.3 (Pin_3), J7.2 (Pin_2), L2.1, Q2.2 (E), R11.1, R12.1, R18.2, R5.2, R6.2, Regulator_Filter1.2, SW2.C, SW2.S2, SW3.2, U10.1 (TEMP), U10.3 (GND), U10.9 (EPAD), U2.4 (Vss), U4.11 (PSN), U4.2 (PGND), U4.21 (CP), U4.25 (EP), U4.3 (PGND), U4.9 (PSP), U5.1 (A1), U5.2 (A0), U5.7 (GND), U6.2 (GND), U7.2 (GND), U8.57 (GND), U9.4 (GND), Y1.2, Y1.4
- net GNDA: now also C2.2, C4.2, D1.2 (A), J2.3 (Pin_3), J4.2 (Pin_2), Q1.3 (S), R21.2, R3.2, R4.2, U11.10 (PB0), U11.4 (VSS), U2.3 (IN-), U3.3 (GND), U4.19 (AGND), U5.9 (Vin-)
- net I2C_SCL: now also U5.5 (SCL), U8.7 (GPIO5)
- net I2C_SDA: now also U5.4 (SDA), U8.6 (GPIO4)
- net Non-inv Input OpAmp: now also R1.2, R3.1, U1.3 (+)
- net POT_SPI_CS: now also U11.1 (~{CS}), U8.15 (GPIO12)
- net POT_SPI_MOSI: now also U11.3 (SI), U8.17 (GPIO14)
- net POT_SPI_SCK: now also U11.2 (SCK), U8.16 (GPIO13)
- net QSPI_CLK: now also U8.52 (QSPI_SCLK), U9.6 (CLK)
- net QSPI_CS: now also U8.56 (QSPI_SS), U9.1 (~{CS})
- net QSPI_IO0: now also U8.53 (QSPI_SD0), U9.5 (DI/IO_{0})
- net QSPI_IO1: now also U8.55 (QSPI_SD1), U9.2 (DO/IO_{1})
- net QSPI_IO2: now also U8.54 (QSPI_SD2), U9.3 (~{WP}/IO_{2})
- net QSPI_IO3: now also U8.51 (QSPI_SD3), U9.7 (~{HOLD}/~{RESET}/IO_{3})
- net RANGE_SELECT: now also Q1.2 (G), U8.9 (GPIO7)
- net ROT_A: now also SW2.A, U8.32 (GPIO21)
- net ROT_B: now also SW2.B, U8.14 (GPIO11)
- net ROT_SW: now also SW2.S1, U8.34 (GPIO22)
- net SWCLK: now also J6.1 (Pin_1), U8.24 (SWCLK)
- net SWD: now also J6.2 (Pin_2), U8.25 (SWD)
- net SWEEP_PWM: now also R22.1, U8.13 (GPIO10)
- net TFT_CS: now also J7.3 (Pin_3), U8.29 (GPIO18)
- net TFT_DC: now also J7.5 (Pin_5), U8.30 (GPIO19)
- net TFT_MISO: now also J7.9 (Pin_9), U8.18 (GPIO15)
- net TFT_MOSI: now also J7.6 (Pin_6), U8.28 (GPIO17)
- net TFT_RST: now also J7.4 (Pin_4), U8.31 (GPIO20)
- net TFT_SCLK: now also J7.7 (Pin_7), U8.27 (GPIO16)
- net USB_DM: now also R15.1, U6.6 (I/O1)
- net USB_DP: now also R14.1, U6.4 (I/O2)
- net USB_D_M: now also R15.2, U8.46 (USB_DM)
- net USB_D_P: now also R14.2, U8.47 (USB_DP)
- net VBUS_SYSTEM: now also C11.1, C3.2, J5.1 (Pin_1), L1.2, U10.5 (BAT), U4.1 (INP), U4.24 (INP), U4.4 (VIN), U4.5 (INN), U4.6 (INN), U7.1 (VIN), U7.3 (EN)
- net V_SWEEP: now also J2.1 (Pin_1), R23.2, U1.7
- net V_filtered: now also C10.1, R22.2, U1.5 (+)
- net Vref: now also C4.1, U11.7 (PA1), U4.17 (VREF)
- net Vref_ADC: now also U2.1 (Vref), U3.2 (OUT)
- net XIN: now also C7.1, U8.20 (XIN), Y1.1
- net XOUT: now also C8.1, U8.21 (XOUT), Y1.3
- net at J1.1 (In): now also SW1.2 (B)
- new net: R21.1, R23.1, U1.6 (-)
- new net: C1.1, SW1.1 (A)
- new net: C1.2, R1.1, SW1.3 (C)
- new net: D2.2 (A), L1.1, U4.7 (BSW)
- new net: Q1.1 (D), R2.2
- new net: D6.1 (K), F1.1
- new net: D4.1 (K), R11.2
- new net: Q2.1 (B), R13.2
- new net: BZ1.2 (-), Q2.3 (C)
- new net: J7.8 (Pin_8), R19.2
- new net: D5.1 (K), R12.2
- new net: R17.2, SW3.1, U8.26 (RUN)
- new net: R20.1, U1.1, U1.2 (-)
- new net: F1.2, FB1.1
- new net: R18.1, U10.2 (PROG)
- new net: D8.1 (K), U10.6 (~{STDBY})
- new net: D7.1 (K), U10.7 (~{CHRG})
- new net: D8.2 (A), R10.2
- new net: D7.2 (A), R9.2
- new net: J3.A5 (CC1), R5.1
- new net: J3.B5 (CC2), R6.1
- new net: D3.1 (K), L2.2, U4.13 (OUTN), U4.14 (OUTN), U4.18 (CN)
Other:
- removed sheet Analog_Frontend
- removed sheet Power_Management
- removed sheet RP2040_Core
- note added: "ANALOG FRONTEND"
- note added: "POWER MANAGEMENT"
- note added: "RP2040 Core"
