File: Auralab_Workstation/analogoscilloscope.kicad_pcb (KiCad board)
At the start: 4 copper layers, 76 parts, among them J1 Conn_Coaxial, J2 TEST_SOCKET, J3 USB_C_Receptacle_USB2.0_16P, J4 Screw_Terminal_01x03, J5 Conn_01x02_Socket, J6 Conn_01x03, J7 Conn_01x14_Socket, Q1 BS170, Q2 BC847, SW1 SW_SPDT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

Commit message: Add files via upload
Parts:
- moved R23 124.1 mm to (172.6, 70.0), turned to 90 degrees
- moved R21 118.0 mm to (166.1, 93.0)
- moved J1 117.0 mm to (149.0, 97.0), turned to 180 degrees
- moved U1 94.4 mm to (149.1, 73.5)
- moved R20 93.4 mm to (136.1, 109.0), turned to 180 degrees
- moved R11 91.5 mm to (148.6, 25.5)
- moved R3 89.7 mm to (137.7, 82.5)
- moved C11 89.6 mm to (159.1, 89.5)
- moved C10 89.5 mm to (155.6, 65.5)
- moved Q1 89.2 mm to (50.3, 119.9)
- moved R4 88.1 mm to (134.2, 50.0), turned to -90 degrees
- moved J4 85.9 mm to (149.6, 57.5), turned to 90 degrees
- moved J2 84.2 mm to (164.1, 62.1), turned to 90 degrees
- moved R1 82.8 mm to (129.6, 82.5)
- moved R8 82.2 mm to (135.6, 57.0)
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Routing:
- net GND: track 229.6 -> 734.1 mm, vias 10 -> 34
- net GNDA: track 20.0 -> 496.5 mm, vias 0 -> 16
- net +3V3_DIGITAL: track 95.7 -> 397.7 mm, vias 9 -> 25
- net /Vref: track 0.00 -> 267.7 mm, vias 0 -> 3
- net VBUS_SYSTEM: track 0.00 -> 232.3 mm, vias 0 -> 15
- net CURRENT_IN: track 0.00 -> 211.0 mm, vias 0 -> 2
- net /+IN_ADC: track 0.00 -> 195.2 mm
- net +5V_RAW: track 0.00 -> 185.9 mm, vias 0 -> 6
- net /FBN: track 0.00 -> 147.4 mm, vias 0 -> 5
- net +Vout: track 0.00 -> 140.3 mm, vias 0 -> 3
- net V_filtered: track 0.00 -> 139.3 mm, vias 0 -> 4
- net -Vout: track 0.00 -> 119.4 mm, vias 0 -> 3
- net Net-(D3-K): track 0.00 -> 93.7 mm, vias 0 -> 2
- net Net-(D2-A): track 0.00 -> 92.4 mm, vias 0 -> 4
- net A6: track 0.00 -> 85.9 mm
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Other:
- board outline added: 154 x 131.5 mm

Commit message: Add files via upload
Routing:
- net GND: track 734.1 -> 736.1 mm
Other:
- board size 154 x 131.5 mm -> 134.5 x 126.5 mm
Changed lines of the file:
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@@
 		(capping no)
 		(filling no)
+		(zone_defaults)
 		(pcbplotparams
 			(layerselection 0x00000000_00000000_55555555_5755f5ff)
@@
 			(at -0.975 -0.975 90)
 			(size 0.5 0.5)
-			(drill 0.2)
+			(drill 0.3)
 			(property pad_prop_heatsink)
 			(layers "*.Cu")
@@
 			(at -0.975 0 90)
 			(size 0.5 0.5)
-			(drill 0.2)
+			(drill 0.3)
 			(property pad_prop_heatsink)
 			(layers "*.Cu")
@@
 			(at -0.975 0.975 90)
 			(size 0.5 0.5)
-			(drill 0.2)
+			(drill 0.3)
 			(property pad_prop_heatsink)
 			(layers "*.Cu")
@@
 			(at 0 -0.975 90)
 			(size 0.5 0.5)
-			(drill 0.2)
+			(drill 0.3)
 			(property pad_prop_heatsink)
 			(layers "*.Cu")
@@
 			(at 0 0 90)
 			(size 0.5 0.5)
-			(drill 0.2)
+			(drill 0.3)
 			(property pad_prop_heatsink)
 			(layers "*.Cu")
@@
 			(at 0 0.975 90)
 			(size 0.5 0.5)
-			(drill 0.2)
+			(drill 0.3)
 			(property pad_prop_heatsink)
 			(layers "*.Cu")
@@
 			(at 0.975 0 90)
 			(size 0.5 0.5)
-			(drill 0.2)
+			(drill 0.3)
 			(property pad_prop_heatsink)
 			(layers "*.Cu")
@@
 			(at 0.975 0.975 90)
 			(size 0.5 0.5)
-			(drill 0.2)
+			(drill 0.3)
 			(property pad_prop_heatsink)
 			(layers "*.Cu")
@@
 			(at -0.7 -1.2)
 			(size 0.5 0.5)
-			(drill 0.2)
+			(drill 0.3)
 			(property pad_prop_heatsink)
 			(layers "*.Cu")
@@
 			(at -0.7 0)
 			(size 0.5 0.5)
-			(drill 0.2)
+			(drill 0.3)
 			(property pad_prop_heatsink)
 			(layers "*.Cu")
@@
 			(at -0.7 1.2)
 			(size 0.5 0.5)
-			(drill 0.2)
+			(drill 0.3)
 			(property pad_prop_heatsink)
 			(layers "*.Cu")
@@
 			(at 0.7 -1.2)
 			(size 0.5 0.5)
-			(drill 0.2)
+			(drill 0.3)
 			(property pad_prop_heatsink)
 			(layers "*.Cu")
@@
 			(at 0.7 0)
 			(size 0.5 0.5)
-			(drill 0.2)
+			(drill 0.3)
 			(property pad_prop_heatsink)
 			(layers "*.Cu")
@@
 			(at 0.7 1.2)
 			(size 0.5 0.5)
-			(drill 0.2)
+			(drill 0.3)
 			(property pad_prop_heatsink)
 			(layers "*.Cu")
@@
 	)
 	(gr_rect
-		(start 25 19)
-		(end 179 150.5)
+		(start 45 21.5)
+		(end 179.5 148)
 		(stroke
 			(width 0.05)
@@
 	)
 	(segment
+		(start 94.5675 67.46)
+		(end 94.180001 67.46)
+		(width 0.2)
+		(layer "F.Cu")
+		(net "GND")
+	)
+	(segment
 		(start 97.18 25.214744)
 		(end 97.18 23.845256)
@@
 	)
 	(segment
+		(start 93.93 67.209999)
+		(end 93.93 66.710001)
+		(width 0.2)
+		(layer "F.Cu")
+		(net "GND")
+	)
+	(segment
 		(start 110.705 50.8)
 		(end 111.555 49.95)
@@
 	)
 	(segment
+		(start 94.180001 66.46)
+		(end 94.5675 66.46)
+		(width 0.2)
+		(layer "F.Cu")
+		(net "GND")
+	)
+	(segment
 		(start 78.6 111.1)
 		(end 77.9 110.4)
@@
 	)
 	(segment
+		(start 94.180001 67.46)
+		(end 93.93 67.209999)
+		(width 0.2)
+		(layer "F.Cu")
+		(net "GND")
+	)
+	(segment
 		(start 111.08 71.057057)
 		(end 113.052943 73.03)
@@
 	)
 	(segment
+		(start 93.93 66.710001)
+		(end 94.180001 66.46)
+		(width 0.2)
+		(layer "F.Cu")
+		(net "GND")
+	)
+	(segment
 		(start 152 33)
 		(end 151.78 32.78)
@@
 		(width 0.2)
 		(layer "B.Cu")
-		(net "+3V3_DIGITAL")
-	)
-	(segment
-		(start 85.03 94.98)
-		(end 85.08 94.93)
-		(width 0.2)
-		(layer "B.Cu")
